File: horizontal/horizontal.kicad_pcb (KiCad board)
At the start: 2 copper layers, 27 x 18.9 mm, 14 parts, among them J2 PROG, J3 Mains, J4 RS485, U1 LM1117-3.3, U2 ESP32-C3-WROOM-02, U4 PSU, U5 MAX485E

Commit message: WIP
Parts:
- removed C1: 10u, Capacitor_SMD:C_0805_2012Metric_Pad1.18x1.45mm_HandSolder
- removed C2, C3: 47u, Capacitor_SMD:C_0805_2012Metric_Pad1.18x1.45mm_HandSolder
- removed C8: 100n, Capacitor_SMD:C_0805_2012Metric_Pad1.18x1.45mm_HandSolder
- removed D1: LED, Connector_PinHeader_2.54mm:PinHeader_1x02_P2.54mm_Vertical
- removed J2: PROG, Connector_PinHeader_2.54mm:PinHeader_1x03_P2.54mm_Vertical
- removed R1: 270R, Resistor_SMD:R_0805_2012Metric_Pad1.20x1.40mm_HandSolder
- removed U1: LM1117-3.3, Package_TO_SOT_SMD:SOT-223-3_TabPin2
- removed U2: ESP32-C3-WROOM-02, Espressif:ESP32-C3-WROOM-02
- removed U5: MAX485E, Package_SO:SO-8_3.9x4.9mm_P1.27mm
- added J1: internal, Connector_PinSocket_2.54mm:PinSocket_1x04_P2.54mm_Vertical, F.Cu at (120.0, 131.0)
- U4: footprint Drake:RQG 5V-0.6A-horizontal sunk -> Drake:RQG 5V-0.6A-vertical
- moved U4 101.9 mm to (90.2, 131.8), turned to -90 degrees
- moved J3 97.0 mm to (79.5, 125.8), turned to -90 degrees
- moved RV1 88.1 mm to (85.5, 127.5), turned to 90 degrees
- moved J4 64.0 mm to (145.5, 131.1), turned to 90 degrees
Routing:
- net Net-(J3-Pin_1): track 0.00 -> 44.5 mm, vias 0 -> 1
- net Net-(J3-Pin_2): track 0.00 -> 35.4 mm, vias 0 -> 1
- net /RS485_B: track 0.00 -> 32.6 mm
- net /RS485_A: track 0.00 -> 28.6 mm
- net GND: vias 0 -> 1
- net +5V: vias 0 -> 2
- added copper zone on F.Cu, net +5V
- added copper zone on B.Cu, net GND
Other:
- board size 27 x 18.9 mm -> 85 x 15 mm
- board text added: "din-rs485-wifi v1.0"

Commit message: WIP
Parts:
- RV1: moved to B.Cu
- moved U4 4.25 mm to (86.0, 131.7)
- moved RV1 2.51 mm to (83.0, 127.8)
Routing:
- net Net-(J3-Pin_1): track 44.5 -> 34.3 mm
- net Net-(J3-Pin_2): track 35.4 -> 26.1 mm

Commit message: WIP
Parts:
- moved U4 21.2 mm to (85.3, 110.5), turned to 180 degrees
- moved J1 2.00 mm to (120.0, 129.0)
Routing:
- net Net-(J3-Pin_1): track 34.3 -> 21.5 mm, vias 1 -> 0
- net Net-(J3-Pin_2): track 26.1 -> 14.8 mm, vias 1 -> 0
- net /RS485_A: track 28.6 -> 26.3 mm
- net /RS485_B: track 32.6 -> 31.1 mm
- net GND: vias 1 -> 0
- net +5V: vias 2 -> 0

Commit message: WIP
Other:
- board text added: "RS485 WiFi v1.0"
- board text removed: "din-rs485-wifi v1.0"
Changed lines of the file:
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@@
   (gr_arc (start 155 134) (mid 154.707107 134.707107) (end 154 135)
     (stroke (width 0.1) (type default)) (layer "Edge.Cuts"))
-  (gr_text "din-rs485-wifi v1.0" (at 116 123) (layer "F.SilkS")
+  (gr_text "RS485 WiFi v1.0" (at 116 123) (layer "F.SilkS")
     (effects (font (size 1.5 1.5) (thickness 0.3) bold) (justify left bottom))
   )

Commit message: WIP
Parts:
- J4: value RS485 -> A RS485 B
- moved J1 7.62 mm to (127.6, 129.0), turned to -90 degrees
Connections:
- J1 pad 1: +5V -> GND
- J1 pad 2: /RS485_B -> /RS485_A
- J1 pad 3: /RS485_A -> /RS485_B
- J1 pad 4: GND -> +5V
Routing:
- net /RS485_A: track 26.3 -> 26.9 mm
Other:
- board text added: "RS485 WiFi v1.1"
- board text removed: "RS485 WiFi v1.0"
Changed lines of the file:
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@@
         (effects (font (size 1 1) (thickness 0.15)))
     )
-    (fp_text value "RS485" (at 3.615 -4 90) (layer "F.SilkS")
+    (fp_text value "A   RS485   B" (at 3.615 -4 90) (layer "F.SilkS")
         (effects (font (size 1 1) (thickness 0.15)))
     )
@@
   )
   (footprint "Connector_PinSocket_2.54mm:PinSocket_1x04_P2.54mm_Vertical" (layer "F.Cu")
-    (at 120 129 90)
+    (at 127.62 129 -90)
     (descr "Through hole straight socket strip, 1x04, 2.54mm pitch, single row (from Kicad 4.0.7), script generated")
     (tags "Through hole socket strip THT 1x04 2.54mm single row")
@@
         (effects (font (size 1 1) (thickness 0.15)))
     )
-    (fp_text value "internal" (at 2.5 1 180) (layer "F.SilkS")
+    (fp_text value "internal" (at 2.5 1) (layer "F.SilkS")
         (effects (font (size 1 1) (thickness 0.15)))
     )
@@
     (fp_line (start 1.27 8.89) (end -1.27 8.89)
       (stroke (width 0.1) (type solid)) (layer "F.Fab"))
-    (pad "1" thru_hole rect (at 0 0 90) (size 1.7 1.7) (drill 1) (layers *.Cu *.Mask)
-      (net 1 "+5V") (pinfunction "Pin_1") (pintype "passive"))
-    (pad "2" thru_hole oval (at 0 2.54 90) (size 1.7 1.7) (drill 1) (layers *.Cu *.Mask)
-      (net 6 "/RS485_B") (pinfunction "Pin_2") (pintype "passive"))
-    (pad "3" thru_hole oval (at 0 5.08 90) (size 1.7 1.7) (drill 1) (layers *.Cu *.Mask)
-      (net 5 "/RS485_A") (pinfunction "Pin_3") (pintype "passive"))
-    (pad "4" thru_hole oval (at 0 7.62 90) (size 1.7 1.7) (drill 1) (layers *.Cu *.Mask)
-      (net 2 "GND") (pinfunction "Pin_4") (pintype "passive"))
+    (pad "1" thru_hole rect (at 0 0 270) (size 1.7 1.7) (drill 1) (layers *.Cu *.Mask)
+      (net 2 "GND") (pinfunction "Pin_1") (pintype "passive"))
+    (pad "2" thru_hole oval (at 0 2.54 270) (size 1.7 1.7) (drill 1) (layers *.Cu *.Mask)
+      (net 5 "/RS485_A") (pinfunction "Pin_2") (pintype "passive"))
+    (pad "3" thru_hole oval (at 0 5.08 270) (size 1.7 1.7) (drill 1) (layers *.Cu *.Mask)
+      (net 6 "/RS485_B") (pinfunction "Pin_3") (pintype "passive"))
+    (pad "4" thru_hole oval (at 0 7.62 270) (size 1.7 1.7) (drill 1) (layers *.Cu *.Mask)
+      (net 1 "+5V") (pinfunction "Pin_4") (pintype "passive"))
     (model "${KICAD6_3DMODEL_DIR}/Connector_PinSocket_2.54mm.3dshapes/PinSocket_1x04_P2.54mm_Vertical.wrl" hide
       (offset (xyz 0 0 0))
@@
     (property "ki_keywords" "VDR resistance")
     (attr smd)
-    (fp_text reference "RV1" (at 0 -2.5 90) (layer "B.SilkS")
+    (fp_text reference "RV1" (at 0 3 90) (layer "B.SilkS")
         (effects (font (size 1 1) (thickness 0.15)) (justify mirror))
     )
@@
   (gr_arc (start 155 134) (mid 154.707107 134.707107) (end 154 135)
     (stroke (width 0.1) (type default)) (layer "Edge.Cuts"))
-  (gr_text "RS485 WiFi v1.0" (at 116 123) (layer "F.SilkS")
+  (gr_text "RS485 WiFi v1.1" (at 116 123) (layer "F.SilkS")
     (effects (font (size 1.5 1.5) (thickness 0.3) bold) (justify left bottom))
   )
@@
   (segment (start 79.5 129.6) (end 85.8615 129.6) (width 1) (layer "B.Cu") (net 4))
   (segment (start 150.500001 131.115) (end 145.500001 131.115) (width 1) (layer "F.Cu") (net 5))
-  (segment (start 127.115 131.115) (end 125.08 129.08) (width 1) (layer "F.Cu") (net 5))
-  (segment (start 145.500001 131.115) (end 127.115 131.115) (width 1) (layer "F.Cu") (net 5))
-  (segment (start 125.08 129.08) (end 125.08 129) (width 1) (layer "F.Cu") (net 5))
+  (segment (start 145.500001 131.115) (end 126.115 131.115) (width 1) (layer "F.Cu") (net 5))
+  (segment (start 125.08 130.08) (end 125.08 129) (width 1) (layer "F.Cu") (net 5))
+  (segment (start 126.115 131.115) (end 125.08 130.08) (width 1) (layer "F.Cu") (net 5))
   (segment (start 150.500001 123.495) (end 145.500001 123.495) (width 1) (layer "F.Cu") (net 6))
+  (segment (start 122.54 127.46) (end 122.54 129) (width 1) (layer "F.Cu") (net 6))
   (segment (start 126.505 123.495) (end 122.54 127.46) (width 1) (layer "F.Cu") (net 6))
   (segment (start 145.500001 123.495) (end 126.505 123.495) (width 1) (layer "F.Cu") (net 6))
-  (segment (start 122.54 127.46) (end 122.54 129) (width 1) (layer "F.Cu") (net 6))
   (zone (net 1) (net_name "+5V") (layer "F.Cu") (hatch edge 0.508)
     (connect_pads (clearance 0.508))
