File: horizontal/horizontal.kicad_sch (KiCad schematic)
At the start: 14 parts, among them J2 PROG, J3 Mains, J4 RS485, U1 LM1117-3.3, U2 ESP32-C3-WROOM-02, U4 PSU, U5 MAX485E

Commit message: WIP
Parts:
- removed C1: 10u, Capacitor_SMD:C_0805_2012Metric_Pad1.18x1.45mm_HandSolder, symbol Device:C
- removed C2, C3: 47u, Capacitor_SMD:C_0805_2012Metric_Pad1.18x1.45mm_HandSolder, symbol Device:C
- removed C8: 100n, Capacitor_SMD:C_0805_2012Metric_Pad1.18x1.45mm_HandSolder, symbol Device:C
- removed D1: LED, Connector_PinHeader_2.54mm:PinHeader_1x02_P2.54mm_Vertical, symbol Device:LED
- removed J2: PROG, Connector_PinHeader_2.54mm:PinHeader_1x03_P2.54mm_Vertical, symbol Connector:Conn_01x03_Female
- removed R1: 270R, Resistor_SMD:R_0805_2012Metric_Pad1.20x1.40mm_HandSolder, symbol Device:R
- removed U1: LM1117-3.3, Package_TO_SOT_SMD:SOT-223-3_TabPin2, symbol Regulator_Linear:LM1117-3.3
- removed U2: ESP32-C3-WROOM-02, Espressif:ESP32-C3-WROOM-02, symbol Espressif:ESP32-C3-WROOM-02
- removed U5: MAX485E, Package_SO:SO-8_3.9x4.9mm_P1.27mm, symbol Interface_UART:MAX485E
- added J1: internal, Connector_PinSocket_2.54mm:PinSocket_1x04_P2.54mm_Vertical, symbol Connector:Conn_01x04_Female
- U4: footprint Drake:RQG 5V-0.6A-horizontal sunk -> Drake:RQG 5V-0.6A-vertical
Connections:
- net +5V: now also J1.1 (Pin_1)
- net GND: now also J1.4 (Pin_4)
- net RS485_A: now also J1.3 (Pin_3)
- net RS485_B: now also J1.2 (Pin_2)
- no-connect marks 9 -> 0
Other:
- moved on the sheet: J3, J4, RV1, U4

Commit message: WIP
Connections:
- net +5V: now also J1.4 (Pin_4); no longer J1.1 (Pin_1)
- net GND: now also J1.1 (Pin_1); no longer J1.4 (Pin_4)
- net RS485_A: now also J1.2 (Pin_2); no longer J1.3 (Pin_3)
- net RS485_B: now also J1.3 (Pin_3); no longer J1.2 (Pin_2)
Changed lines of the file:
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@@
-(kicad_sch (version 20221004) (generator eeschema)
+(kicad_sch (version 20221126) (generator eeschema)
   (paper "A4")
   (junction (at 93.98 76.2) (diameter 0) (color 0 0 0 0)
@@
       (project "horizontal"
         (path "/32f9e9f8-9d15-4d51-acc1-705de5fd2b71"
-          (reference "U4") (unit 1) (value "PSU") (footprint "Drake:RQG 5V-0.6A-vertical")
+          (reference "U4") (unit 1)
         )
       )
@@
       (project "horizontal"
         (path "/32f9e9f8-9d15-4d51-acc1-705de5fd2b71"
-          (reference "#PWR03") (unit 1) (value "GND") (footprint "")
+          (reference "#PWR03") (unit 1)
         )
       )
@@
       (project "horizontal"
         (path "/32f9e9f8-9d15-4d51-acc1-705de5fd2b71"
-          (reference "J4") (unit 1) (value "RS485") (footprint "Drake:DG235-3.81-03P")
+          (reference "J4") (unit 1)
         )
       )
@@
       (project "horizontal"
         (path "/32f9e9f8-9d15-4d51-acc1-705de5fd2b71"
-          (reference "#PWR0106") (unit 1) (value "+5V") (footprint "")
-        )
-      )
-    )
-  )
-  (symbol (lib_id "Connector:Conn_01x04_Female") (at 161.29 102.87 0) (unit 1)
-    (in_bom yes) (on_board yes) (dnp no) (fields_autoplaced)
-    (property "Reference" "J1" (at 162.0012 103.5455 0)
-      (effects (font (size 1.27 1.27)) (justify left))
-    )
-    (property "Value" "internal" (at 162.0012 105.3077 0)
-      (effects (font (size 1.27 1.27)) (justify left))
-    )
-    (property "Footprint" "Connector_PinSocket_2.54mm:PinSocket_1x04_P2.54mm_Vertical" (at 161.29 102.87 0)
-      (effects (font (size 1.27 1.27)) hide)
-    )
-    (property "Datasheet" "~" (at 161.29 102.87 0)
+          (reference "#PWR0106") (unit 1)
+        )
+      )
+    )
+  )
+  (symbol (lib_id "Connector:Conn_01x04_Female") (at 161.29 105.41 0) (mirror x) (unit 1)
+    (in_bom yes) (on_board yes) (dnp no)
+    (property "Reference" "J1" (at 162.0012 104.7345 0)
+      (effects (font (size 1.27 1.27)) (justify left))
+    )
+    (property "Value" "internal" (at 162.0012 102.9723 0)
+      (effects (font (size 1.27 1.27)) (justify left))
+    )
+    (property "Footprint" "Connector_PinSocket_2.54mm:PinSocket_1x04_P2.54mm_Vertical" (at 161.29 105.41 0)
+      (effects (font (size 1.27 1.27)) hide)
+    )
+    (property "Datasheet" "~" (at 161.29 105.41 0)
       (effects (font (size 1.27 1.27)) hide)
     )
@@
       (project "horizontal"
         (path "/32f9e9f8-9d15-4d51-acc1-705de5fd2b71"
-          (reference "J1") (unit 1) (value "internal") (footprint "Connector_PinSocket_2.54mm:PinSocket_1x04_P2.54mm_Vertical")
+          (reference "J1") (unit 1)
         )
       )
@@
       (project "horizontal"
         (path "/32f9e9f8-9d15-4d51-acc1-705de5fd2b71"
-          (reference "J3") (unit 1) (value "Mains") (footprint "Drake:DG235-3.81-02P")
+          (reference "J3") (unit 1)
         )
       )
@@
       (project "horizontal"
         (path "/32f9e9f8-9d15-4d51-acc1-705de5fd2b71"
-          (reference "RV1") (unit 1) (value "B72650M251K72") (footprint "Resistor_SMD:R_1210_3225Metric_Pad1.30x2.65mm_HandSolder")
+          (reference "RV1") (unit 1)
         )
       )
@@
   )
   (sheet_instances
-    (path "/32f9e9f8-9d15-4d51-acc1-705de5fd2b71" (page "1"))
+    (path "/" (page "1"))
   )
 )
