File: vertical/vertical.kicad_pcb (KiCad board)
At the start: 2 copper layers, 27 x 18.9 mm, 14 parts, among them J2 PROG, J3 Mains, J4 RS485, U1 LM1117-3.3, U2 ESP32-C3-WROOM-02, U4 PSU, U5 MAX485E

Commit message: WIP
Parts:
- removed J3: Mains, Drake:DG235-3.81-02P
- removed J4: RS485, Drake:DG235-3.81-03P
- removed RV1: B72650M251K72, Resistor_SMD:R_1210_3225Metric_Pad1.30x2.65mm_HandSolder
- removed U4: PSU, Drake:RQG 5V-0.6A-horizontal sunk
- added J1: internal, Connector_PinHeader_2.54mm:PinHeader_1x04_P2.54mm_Vertical, F.Cu at (174.8, 88.7)
- moved D1 32.9 mm to (162.5, 111.3)
- moved U5 32.9 mm to (155.9, 112.2)
- moved J2 15.6 mm to (174.8, 109.2)
- moved U1 12.5 mm to (177.3, 102.8)
- moved U2 10.9 mm to (162.1, 99.0)
- moved C1 10.7 mm to (179.5, 87.9)
- moved C3 10.7 mm to (179.5, 93.9)
- moved C8 10.7 mm to (179.5, 96.9)
- moved C2 10.7 mm to (179.5, 90.9)
- moved R1 7.57 mm to (167.2, 110.5)
Other:
- board outline removed

Commit message: WIP
Parts:
- added R2: 270R, Resistor_SMD:R_0805_2012Metric_Pad1.20x1.40mm_HandSolder, F.Cu at (141.0, 85.0)
- added R3: 270R, Resistor_SMD:R_0805_2012Metric_Pad1.20x1.40mm_HandSolder, F.Cu at (141.0, 81.0)
- added R4: 270R, Resistor_SMD:R_0805_2012Metric_Pad1.20x1.40mm_HandSolder, F.Cu at (141.0, 83.0)
- C1, C2, C3, R1, U1: moved to B.Cu
- D1: footprint Connector_PinHeader_2.54mm:PinHeader_1x02_P2.54mm_Vertical -> LED_SMD:LED_2010_5025Metric; moved to B.Cu
- J1: footprint Connector_PinHeader_2.54mm:PinHeader_1x04_P2.54mm_Vertical -> Connector_PinHeader_2.54mm:PinHeader_1x04_P2.54mm_Horizontal
- moved J2 61.5 mm to (127.0, 70.5)
- moved C8 52.5 mm to (128.5, 84.5), turned to 180 degrees
- moved U1 51.5 mm to (130.0, 82.5), turned to 180 degrees
- moved C1 49.5 mm to (130.0, 88.0), turned to 180 degrees
- moved D1 44.9 mm to (147.5, 69.0), turned to -90 degrees
- moved C2 44.0 mm to (136.5, 81.5), turned to 90 degrees
- moved C3 42.3 mm to (139.0, 81.5), turned to 90 degrees
- moved R1 40.6 mm to (147.5, 75.0), turned to 90 degrees
- moved U2 36.4 mm to (140.0, 70.0)
- moved U5 36.0 mm to (135.0, 83.0), turned to 180 degrees
- moved J1 33.5 mm to (141.3, 88.0), turned to -90 degrees
Connections:
- C8 pad 1: +3V3 -> +5V
- U2 pad 11: /RX -> Net-(U2-GPIO20/U0RXD)
- U2 pad 12: /TX -> Net-(U2-GPIO21/U0TXD)
- U2 pad 15: /TXEN -> Net-(U2-GPIO3/ADC1_CH3)
- U5 pad 8: +3V3 -> +5V
Routing:
- net GND: track 0.00 -> 42.6 mm, vias 0 -> 9
- net /USB_D-: track 0.00 -> 27.7 mm, vias 0 -> 1
- net /LED: track 0.00 -> 26.8 mm, vias 0 -> 1
- net /USB_D+: track 0.00 -> 26.2 mm, vias 0 -> 1
- net Net-(U2-GPIO3/ADC1_CH3): track 0.00 -> 17.2 mm
- net +5V: track 0.00 -> 15.9 mm
- net Net-(U2-GPIO20/U0RXD): track 0.00 -> 13.8 mm
- net Net-(U2-GPIO21/U0TXD): track 0.00 -> 10.8 mm
- net /RS485_A: track 0.00 -> 9.98 mm
- net +3V3: track 0.00 -> 6.81 mm, vias 0 -> 4
- net /RS485_B: track 0.00 -> 6.65 mm
- net /TXEN: track 0.00 -> 3.73 mm
- net Net-(D1-A): track 0.00 -> 2.75 mm
- net /TX: track 0.00 -> 2.46 mm
- net /RX: track 0.00 -> 2.46 mm
- added copper zone on B.Cu, net +3V3
- added copper zone on F.Cu, net GND
Other:
- board outline added: 25 x 25 mm

Commit message: WIP
Other:
- board text added: "EDA&TATA"
- board text added: "RS485 WiFi v1.0"
Changed lines of the file:
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@@
   (setup
     (stackup
-      (layer "F.SilkS" (type "Top Silk Screen"))
+      (layer "F.SilkS" (type "Top Silk Screen") (color "White"))
       (layer "F.Paste" (type "Top Solder Paste"))
-      (layer "F.Mask" (type "Top Solder Mask") (thickness 0.01))
+      (layer "F.Mask" (type "Top Solder Mask") (color "Blue") (thickness 0.01))
       (layer "F.Cu" (type "copper") (thickness 0.035))
       (layer "dielectric 1" (type "core") (thickness 1.51) (material "FR4") (epsilon_r 4.5) (loss_tangent 0.02))
       (layer "B.Cu" (type "copper") (thickness 0.035))
-      (layer "B.Mask" (type "Bottom Solder Mask") (thickness 0.01))
+      (layer "B.Mask" (type "Bottom Solder Mask") (color "Blue") (thickness 0.01))
       (layer "B.Paste" (type "Bottom Solder Paste"))
-      (layer "B.SilkS" (type "Bottom Silk Screen"))
+      (layer "B.SilkS" (type "Bottom Silk Screen") (color "White"))
       (copper_finish "None")
       (dielectric_constraints no)
@@
     (fp_line (start 1 0.625) (end -1 0.625)
       (stroke (width 0.1) (type solid)) (layer "F.Fab"))
-    (pad "1" smd roundrect (at -1 0 180) (size 1.2 1.4) (layers "F.Cu" "F.Paste" "F.Mask") (roundrect_rratio 0.208333)
+    (pad "1" smd roundrect (at -1 0 180) (size 1.2 1.4) (layers "F.Cu" "F.Paste" "F.Mask") (roundrect_rratio 0.2083333333)
       (net 23 "Net-(U2-GPIO21{slash}U0TXD)") (pintype "passive"))
-    (pad "2" smd roundrect (at 1 0 180) (size 1.2 1.4) (layers "F.Cu" "F.Paste" "F.Mask") (roundrect_rratio 0.208333)
+    (pad "2" smd roundrect (at 1 0 180) (size 1.2 1.4) (layers "F.Cu" "F.Paste" "F.Mask") (roundrect_rratio 0.2083333333)
       (net 19 "/TX") (pintype "passive"))
     (model "${KICAD6_3DMODEL_DIR}/Resistor_SMD.3dshapes/R_0805_2012Metric.wrl"
@@
     (fp_line (start 1 0.625) (end -1 0.625)
       (stroke (width 0.1) (type solid)) (layer "F.Fab"))
-    (pad "1" smd roundrect (at -1 0) (size 1.2 1.4) (layers "F.Cu" "F.Paste" "F.Mask") (roundrect_rratio 0.208333)
+    (pad "1" smd roundrect (at -1 0) (size 1.2 1.4) (layers "F.Cu" "F.Paste" "F.Mask") (roundrect_rratio 0.2083333333)
       (net 20 "/TXEN") (pintype "passive"))
-    (pad "2" smd roundrect (at 1 0) (size 1.2 1.4) (layers "F.Cu" "F.Paste" "F.Mask") (roundrect_rratio 0.208333)
+    (pad "2" smd roundrect (at 1 0) (size 1.2 1.4) (layers "F.Cu" "F.Paste" "F.Mask") (roundrect_rratio 0.2083333333)
       (net 24 "Net-(U2-GPIO3{slash}ADC1_CH3)") (pintype "passive"))
     (model "${KICAD6_3DMODEL_DIR}/Resistor_SMD.3dshapes/R_0805_2012Metric.wrl"
@@
     (fp_line (start 1 0.625) (end -1 0.625)
       (stroke (width 0.1) (type solid)) (layer "F.Fab"))
-    (pad "1" smd roundrect (at -1.0375 0 180) (size 1.175 1.45) (layers "F.Cu" "F.Paste" "F.Mask") (roundrect_rratio 0.212766)
+    (pad "1" smd roundrect (at -1.0375 0 180) (size 1.175 1.45) (layers "F.Cu" "F.Paste" "F.Mask") (roundrect_rratio 0.2127659574)
       (net 1 "+5V") (pintype "passive"))
-    (pad "2" smd roundrect (at 1.0375 0 180) (size 1.175 1.45) (layers "F.Cu" "F.Paste" "F.Mask") (roundrect_rratio 0.212766)
+    (pad "2" smd roundrect (at 1.0375 0 180) (size 1.175 1.45) (layers "F.Cu" "F.Paste" "F.Mask") (roundrect_rratio 0.2127659574)
       (net 2 "GND") (pintype "passive"))
     (model "${KICAD6_3DMODEL_DIR}/Capacitor_SMD.3dshapes/C_0805_2012Metric.wrl"
@@
     (fp_line (start 1 0.625) (end -1 0.625)
       (stroke (width 0.1) (type solid)) (layer "F.Fab"))
-    (pad "1" smd roundrect (at -1 0 180) (size 1.2 1.4) (layers "F.Cu" "F.Paste" "F.Mask") (roundrect_rratio 0.208333)
+    (pad "1" smd roundrect (at -1 0 180) (size 1.2 1.4) (layers "F.Cu" "F.Paste" "F.Mask") (roundrect_rratio 0.2083333333)
       (net 22 "Net-(U2-GPIO20{slash}U0RXD)") (pintype "passive"))
-    (pad "2" smd roundrect (at 1 0 180) (size 1.2 1.4) (layers "F.Cu" "F.Paste" "F.Mask") (roundrect_rratio 0.208333)
+    (pad "2" smd roundrect (at 1 0 180) (size 1.2 1.4) (layers "F.Cu" "F.Paste" "F.Mask") (roundrect_rratio 0.2083333333)
       (net 18 "/RX") (pintype "passive"))
     (model "${KICAD6_3DMODEL_DIR}/Resistor_SMD.3dshapes/R_0805_2012Metric.wrl"
@@
     (fp_line (start 1 0.625) (end 1 -0.625)
       (stroke (width 0.1) (type solid)) (layer "B.Fab"))
-    (pad "1" smd roundrect (at -1.0375 0 90) (size 1.175 1.45) (layers "B.Cu" "B.Paste" "B.Mask") (roundrect_rratio 0.212766)
+    (pad "1" smd roundrect (at -1.0375 0 90) (size 1.175 1.45) (layers "B.Cu" "B.Paste" "B.Mask") (roundrect_rratio 0.2127659574)
       (net 3 "+3V3") (pintype "passive"))
-    (pad "2" smd roundrect (at 1.0375 0 90) (size 1.175 1.45) (layers "B.Cu" "B.Paste" "B.Mask") (roundrect_rratio 0.212766)
+    (pad "2" smd roundrect (at 1.0375 0 90) (size 1.175 1.45) (layers "B.Cu" "B.Paste" "B.Mask") (roundrect_rratio 0.2127659574)
       (net 2 "GND") (pintype "passive"))
     (model "${KICAD6_3DMODEL_DIR}/Capacitor_SMD.3dshapes/C_0805_2012Metric.wrl"
@@
     (fp_line (start 1 0.625) (end 1 -0.625)
       (stroke (width 0.1) (type solid)) (layer "B.Fab"))
-    (pad "1" smd roundrect (at -1.0375 0 90) (size 1.175 1.45) (layers "B.Cu" "B.Paste" "B.Mask") (roundrect_rratio 0.212766)
+    (pad "1" smd roundrect (at -1.0375 0 90) (size 1.175 1.45) (layers "B.Cu" "B.Paste" "B.Mask") (roundrect_rratio 0.2127659574)
       (net 3 "+3V3") (pintype "passive"))
-    (pad "2" smd roundrect (at 1.0375 0 90) (size 1.175 1.45) (layers "B.Cu" "B.Paste" "B.Mask") (roundrect_rratio 0.212766)
+    (pad "2" smd roundrect (at 1.0375 0 90) (size 1.175 1.45) (layers "B.Cu" "B.Paste" "B.Mask") (roundrect_rratio 0.2127659574)
       (net 2 "GND") (pintype "passive"))
     (model "${KICAD6_3DMODEL_DIR}/Capacitor_SMD.3dshapes/C_0805_2012Metric.wrl"
@@
     (fp_line (start 2.5 1.25) (end -1.875 1.25)
       (stroke (width 0.1) (type solid)) (layer "B.Fab"))
-    (pad "1" smd roundrect (at -2.25 0 270) (size 1.35 2.65) (layers "B.Cu" "B.Paste" "B.Mask") (roundrect_rratio 0.185185)
+    (pad "1" smd roundrect (at -2.25 0 270) (size 1.35 2.65) (layers "B.Cu" "B.Paste" "B.Mask") (roundrect_rratio 0.1851851852)
       (net 2 "GND") (pinfunction "K") (pintype "passive"))
-    (pad "2" smd roundrect (at 2.25 0 270) (size 1.35 2.65) (layers "B.Cu" "B.Paste" "B.Mask") (roundrect_rratio 0.185185)
+    (pad "2" smd roundrect (at 2.25 0 270) (size 1.35 2.65) (layers "B.Cu" "B.Paste" "B.Mask") (roundrect_rratio 0.1851851852)
       (net 9 "Net-(D1-A)") (pinfunction "A") (pintype "passive"))
     (model "${KICAD6_3DMODEL_DIR}/LED_SMD.3dshapes/LED_2010_5025Metric.wrl" hide
@@
     (fp_line (start 1 0.625) (end 1 -0.625)
       (stroke (width 0.1) (type solid)) (layer "B.Fab"))
-    (pad "1" smd roundrect (at -1 0 90) (size 1.2 1.4) (layers "B.Cu" "B.Paste" "B.Mask") (roundrect_rratio 0.208333)
+    (pad "1" smd roundrect (at -1 0 90) (size 1.2 1.4) (layers "B.Cu" "B.Paste" "B.Mask") (roundrect_rratio 0.2083333333)
       (net 21 "/LED") (pintype "passive"))
-    (pad "2" smd roundrect (at 1 0 90) (size 1.2 1.4) (layers "B.Cu" "B.Paste" "B.Mask") (roundrect_rratio 0.208333)
+    (pad "2" smd roundrect (at 1 0 90) (size 1.2 1.4) (layers "B.Cu" "B.Paste" "B.Mask") (roundrect_rratio 0.2083333333)
       (net 9 "Net-(D1-A)") (pintype "passive"))
     (model "${KICAD6_3DMODEL_DIR}/Resistor_SMD.3dshapes/R_0805_2012Metric.wrl"
@@
     (fp_line (start 1 0.625) (end 1 -0.625)
       (stroke (width 0.1) (type solid)) (layer "B.Fab"))
-    (pad "1" smd roundrect (at -1.0375 0 180) (size 1.175 1.45) (layers "B.Cu" "B.Paste" "B.Mask") (roundrect_rratio 0.212766)
+    (pad "1" smd roundrect (at -1.0375 0 180) (size 1.175 1.45) (layers "B.Cu" "B.Paste" "B.Mask") (roundrect_rratio 0.2127659574)
       (net 1 "+5V") (pintype "passive"))
-    (pad "2" smd roundrect (at 1.0375 0 180) (size 1.175 1.45) (layers "B.Cu" "B.Paste" "B.Mask") (roundrect_rratio 0.212766)
+    (pad "2" smd roundrect (at 1.0375 0 180) (size 1.175 1.45) (layers "B.Cu" "B.Paste" "B.Mask") (roundrect_rratio 0.2127659574)
       (net 2 "GND") (pintype "passive"))
     (model "${KICAD6_3DMODEL_DIR}/Capacitor_SMD.3dshapes/C_0805_2012Metric.wrl"
@@
     )
   )
+  (gr_line (start 147 81) (end 147 90)
+    (stroke (width 0.15) (type default)) (layer "F.SilkS"))
+  (gr_line (start 150 81) (end 147 81)
+    (stroke (width 0.15) (type default)) (layer "F.SilkS"))
+  (gr_line (start 150 81) (end 150 90)
+    (stroke (width 0.15) (type default)) (layer "F.SilkS"))
+  (gr_line (start 150 90) (end 147 90)
+    (stroke (width 0.15) (type default)) (layer "F.SilkS"))
   (gr_line (start 125 90) (end 150 90)
     (stroke (width 0.1) (type default)) (layer "Edge.Cuts"))
@@
   (gr_line (start 150 65) (end 125 65)
     (stroke (width 0.1) (type default)) (layer "Edge.Cuts"))
+  (gr_text "RS485 WiFi v1.0" (at 126 80) (layer "F.SilkS")
+    (effects (font (size 0.8 0.8) (thickness 0.2) bold) (justify left bottom))
+  )
+  (gr_text "EDA&TATA" (at 149 89 90) (layer "F.SilkS")
+    (effects (font (size 1 1) (thickness 0.25) bold) (justify left bottom))
+  )
   (dimension (type aligned) (layer "Dwgs.User")
     (pts (xy 125 65) (xy 137.5 65))

Commit message: WIP
Parts:
- moved D1 19.1 mm to (128.5, 67.0), turned to 0 degrees
- moved R1 14.6 mm to (135.0, 67.5)
Routing:
- net /LED: track 26.8 -> 4.02 mm
- net GND: track 42.6 -> 23.1 mm
- net /USB_D-: track 27.7 -> 25.0 mm
- net +3V3: track 6.81 -> 8.93 mm, vias 4 -> 1
- net Net-(D1-A): track 2.75 -> 4.46 mm
Other:
- board text added: "RS485 WiFi v1.1"
- board text removed: "RS485 WiFi v1.0"
