File: vertical/vertical.kicad_sch (KiCad schematic)
At the start: 14 parts, among them J2 PROG, J3 Mains, J4 RS485, U1 LM1117-3.3, U2 ESP32-C3-WROOM-02, U4 PSU, U5 MAX485E

Commit message: WIP
Parts:
- removed J3: Mains, Drake:DG235-3.81-02P, symbol Connector:Conn_01x02_Female
- removed J4: RS485, Drake:DG235-3.81-03P, symbol Connector:Conn_01x03_Female
- removed RV1: B72650M251K72, Resistor_SMD:R_1210_3225Metric_Pad1.30x2.65mm_HandSolder, symbol Device:Varistor
- removed U4: PSU, Drake:RQG 5V-0.6A-horizontal sunk, symbol Drake:PSU
- added J1: internal, Connector_PinHeader_2.54mm:PinHeader_1x04_P2.54mm_Vertical, symbol Connector:Conn_01x04_Male
Connections:
- net +5V: now also J1.4 (Pin_4)
- net GND: now also J1.1 (Pin_1)
- net RS485_A: now also J1.2 (Pin_2)
- net RS485_B: now also J1.3 (Pin_3)
Changed lines of the file:
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@@
 (kicad_sch (version 20221004) (generator eeschema)
   (paper "A4")
-  (junction (at 60.96 55.88) (diameter 0) (color 0 0 0 0)
-  )
-  (junction (at 60.96 63.5) (diameter 0) (color 0 0 0 0)
-  )
   (junction (at 81.28 82.55) (diameter 0) (color 0 0 0 0)
   )
@@
     (stroke (width 0) (type default))
   )
-  (wire (pts (xy 52.07 63.5) (xy 60.96 63.5))
-    (stroke (width 0) (type default))
-  )
   (wire (pts (xy 91.44 82.55) (xy 91.44 83.82))
     (stroke (width 0) (type default))
   )
-  (wire (pts (xy 60.96 63.5) (xy 71.12 63.5))
-    (stroke (width 0) (type default))
-  )
-  (wire (pts (xy 60.96 55.88) (xy 71.12 55.88))
-    (stroke (width 0) (type default))
-  )
   (wire (pts (xy 104.14 123.19) (xy 107.95 123.19))
     (stroke (width 0) (type default))
@@
     (stroke (width 0) (type default))
   )
-  (wire (pts (xy 52.07 55.88) (xy 60.96 55.88))
-    (stroke (width 0) (type default))
-  )
   (wire (pts (xy 49.53 82.55) (xy 54.61 82.55))
     (stroke (width 0) (type default))
   )
   (wire (pts (xy 91.44 82.55) (xy 96.52 82.55))
-    (stroke (width 0) (type default))
-  )
-  (wire (pts (xy 52.07 58.42) (xy 52.07 63.5))
     (stroke (width 0) (type default))
   )
@@
     (effects (font (size 1.27 1.27)) (justify left bottom))
   )
-  (label "RS485_B" (at 229.87 74.93 180) (fields_autoplaced)
+  (label "RS485_B" (at 184.15 125.73 180) (fields_autoplaced)
     (effects (font (size 1.27 1.27)) (justify right bottom))
   )
@@
     (effects (font (size 1.27 1.27)) (justify right bottom))
   )
+  (label "+5V" (at 184.15 123.19 180) (fields_autoplaced)
+    (effects (font (size 1.27 1.27)) (justify right bottom))
+  )
   (label "LED" (at 134.62 71.12 180) (fields_autoplaced)
     (effects (font (size 1.27 1.27)) (justify right bottom))
@@
     (effects (font (size 1.27 1.27)) (justify right bottom))
   )
-  (label "GND" (at 229.87 72.39 180) (fields_autoplaced)
+  (label "GND" (at 184.15 130.81 180) (fields_autoplaced)
+    (effects (font (size 1.27 1.27)) (justify right bottom))
+  )
+  (label "RS485_A" (at 184.15 128.27 180) (fields_autoplaced)
     (effects (font (size 1.27 1.27)) (justify right bottom))
   )
@@
     (effects (font (size 1.27 1.27)) (justify left bottom))
   )
-  (label "RS485_A" (at 229.87 69.85 180) (fields_autoplaced)
-    (effects (font (size 1.27 1.27)) (justify right bottom))
-  )
   (label "TX" (at 93.98 143.51 180) (fields_autoplaced)
     (effects (font (size 1.27 1.27)) (justify right bottom))
@@
         (path "/32f9e9f8-9d15-4d51-acc1-705de5fd2b71"
           (reference "C3") (unit 1) (value "47u") (footprint "Capacitor_SMD:C_0805_2012Metric_Pad1.18x1.45mm_HandSolder")
-        )
-      )
-    )
-  )
-  (symbol (lib_id "Drake:PSU") (at 83.82 59.69 0) (unit 1)
-    (in_bom yes) (on_board yes) (dnp no) (fields_autoplaced)
-    (property "Reference" "U4" (at 83.82 50.2971 0)
-      (effects (font (size 1.524 1.524)))
-    )
-    (property "Value" "PSU" (at 83.82 52.3609 0)
-      (effects (font (size 1.524 1.524)))
-    )
-    (property "Footprint" "Drake:RQG 5V-0.6A-horizontal sunk" (at 83.82 59.69 0)
-      (effects (font (size 1.524 1.524)) hide)
-    )
-    (property "Datasheet" "" (at 83.82 59.69 0)
-      (effects (font (size 1.524 1.524)) hide)
-    )
-    (pin "1")
-    (pin "2")
-    (pin "3")
-    (pin "4")
-    (instances
-      (project "vertical"
-        (path "/32f9e9f8-9d15-4d51-acc1-705de5fd2b71"
-          (reference "U4") (unit 1) (value "PSU") (footprint "Drake:RQG 5V-0.6A-horizontal sunk")
         )
       )
@@
     )
   )
-  (symbol (lib_id "power:GND") (at 96.52 63.5 0) (unit 1)
-    (in_bom yes) (on_board yes) (dnp no) (fields_autoplaced)
-    (property "Reference" "#PWR03" (at 96.52 69.85 0)
-      (effects (font (size 1.27 1.27)) hide)
-    )
-    (property "Value" "GND" (at 96.52 67.5561 0)
-      (effects (font (size 1.27 1.27)))
-    )
-    (property "Footprint" "" (at 96.52 63.5 0)
-      (effects (font (size 1.27 1.27)) hide)
-    )
-    (property "Datasheet" "" (at 96.52 63.5 0)
-      (effects (font (size 1.27 1.27)) hide)
-    )
-    (pin "1")
-    (instances
-      (project "vertical"
-        (path "/32f9e9f8-9d15-4d51-acc1-705de5fd2b71"
-          (reference "#PWR03") (unit 1) (value "GND") (footprint "")
-        )
-      )
-    )
-  )
-  (symbol (lib_id "Connector:Conn_01x03_Female") (at 234.95 72.39 0) (unit 1)
-    (in_bom yes) (on_board yes) (dnp no) (fields_autoplaced)
-    (property "Reference" "J4" (at 235.6612 71.7955 0)
-      (effects (font (size 1.27 1.27)) (justify left))
-    )
-    (property "Value" "RS485" (at 235.6612 73.5577 0)
-      (effects (font (size 1.27 1.27)) (justify left))
-    )
-    (property "Footprint" "Drake:DG235-3.81-03P" (at 234.95 72.39 0)
-      (effects (font (size 1.27 1.27)) hide)
-    )
-    (property "Datasheet" "~" (at 234.95 72.39 0)
+  (symbol (lib_id "Connector:Conn_01x04_Male") (at 189.23 128.27 180) (unit 1)
+    (in_bom yes) (on_board yes) (dnp no) (fields_autoplaced)
+    (property "Reference" "J1" (at 189.9412 126.4055 0)
+      (effects (font (size 1.27 1.27)) (justify right))
+    )
+    (property "Value" "internal" (at 189.9412 128.1677 0)
+      (effects (font (size 1.27 1.27)) (justify right))
+    )
+    (property "Footprint" "Connector_PinHeader_2.54mm:PinHeader_1x04_P2.54mm_Vertical" (at 189.23 128.27 0)
+      (effects (font (size 1.27 1.27)) hide)
+    )
+    (property "Datasheet" "~" (at 189.23 128.27 0)
       (effects (font (size 1.27 1.27)) hide)
     )
@@
     (pin "2")
     (pin "3")
-    (instances
-      (project "vertical"
-        (path "/32f9e9f8-9d15-4d51-acc1-705de5fd2b71"
-          (reference "J4") (unit 1) (value "RS485") (footprint "Drake:DG235-3.81-03P")
+    (pin "4")
+    (instances
+      (project "vertical"
+        (path "/32f9e9f8-9d15-4d51-acc1-705de5fd2b71"
+          (reference "J1") (unit 1) (value "internal") (footprint "Connector_PinHeader_2.54mm:PinHeader_1x04_P2.54mm_Vertical")
         )
       )
@@
         (path "/32f9e9f8-9d15-4d51-acc1-705de5fd2b71"
           (reference "#PWR0105") (unit 1) (value "GND") (footprint "")
-        )
-      )
-    )
-  )
-  (symbol (lib_id "power:+5V") (at 96.52 55.88 270) (unit 1)
-    (in_bom yes) (on_board yes) (dnp no) (fields_autoplaced)
-    (property "Reference" "#PWR0106" (at 92.71 55.88 0)
-      (effects (font (size 1.27 1.27)) hide)
-    )
-    (property "Value" "+5V" (at 99.695 56.1666 90)
-      (effects (font (size 1.27 1.27)) (justify left))
-    )
-    (property "Footprint" "" (at 96.52 55.88 0)
-      (effects (font (size 1.27 1.27)) hide)
-    )
-    (property "Datasheet" "" (at 96.52 55.88 0)
-      (effects (font (size 1.27 1.27)) hide)
-    )
-    (pin "1")
-    (instances
-      (project "vertical"
-        (path "/32f9e9f8-9d15-4d51-acc1-705de5fd2b71"
-          (reference "#PWR0106") (unit 1) (value "+5V") (footprint "")
         )
       )
@@
         )
       )
-    )
-  )
-  (symbol (lib_id "Connector:Conn_01x02_Female") (at 46.99 58.42 180) (unit 1)
-    (in_bom yes) (on_board yes) (dnp no)
-    (property "Reference" "J3" (at 46.99 53.34 0)
-      (effects (font (size 1.27 1.27)))
-    )
-    (property "Value" "Mains" (at 46.99 60.96 0)
-      (effects (font (size 1.27 1.27)))
-    )
-    (property "Footprint" "Drake:DG235-3.81-02P" (at 46.99 58.42 0)
-      (effects (font (size 1.27 1.27)) hide)
-    )
-    (property "Datasheet" "~" (at 46.99 58.42 0)
-      (effects (font (size 1.27 1.27)) hide)
-    )
-    (pin "1")
-    (pin "2")
-    (instances
-      (project "vertical"
-        (path "/32f9e9f8-9d15-4d51-acc1-705de5fd2b71"
-          (reference "J3") (unit 1) (value "Mains") (footprint "Drake:DG235-3.81-02P")
-        )
-      )
-    )
-  )
-  (symbol (lib_id "Device:Varistor") (at 60.96 59.69 0) (unit 1)
-    (in_bom yes) (on_board yes) (dnp no)
-    (property "Reference" "RV1" (at 63.4999 59.155 0)
-      (effects (font (size 1.27 1.27)) (justify left))
-    )
-    (property "Value" "B72650M251K72" (at 53.34 66.04 0)
-      (effects (font (size 1.27 1.27)) (justify left))
-    )
-    (property "Footprint" "Resistor_SMD:R_1210_3225Metric_Pad1.30x2.65mm_HandSolder" (at 59.182 59.69 90)
-      (effects (font (size 1.27 1.27)) hide)
-    )
-    (property "Datasheet" "~" (at 60.96 59.69 0)
-      (effects (font (size 1.27 1.27)) hide)
-    )
-    (pin "1")
-    (pin "2")
-    (instances
-      (project "vertical"
-        (path "/32f9e9f8-9d15-4d51-acc1-705de5fd2b71"
-          (reference "RV1") (unit 1) (value "B72650M251K72") (footprint "Resistor_SMD:R_1210_3225Metric_Pad1.30x2.65mm_HandSolder")
-        )
-      )

Commit message: WIP
Parts:
- added R2, R3, R4: 270R, Resistor_SMD:R_0805_2012Metric_Pad1.20x1.40mm_HandSolder, symbol Device:R
- D1: footprint Connector_PinHeader_2.54mm:PinHeader_1x02_P2.54mm_Vertical -> LED_SMD:LED_2010_5025Metric
- J1: footprint Connector_PinHeader_2.54mm:PinHeader_1x04_P2.54mm_Vertical -> Connector_PinHeader_2.54mm:PinHeader_1x04_P2.54mm_Horizontal
Connections:
- net +3V3: no longer C8.1, U5.8 (VCC)
- net +5V: now also C8.1, U5.8 (VCC)
- net RX: now also R2.2; no longer U2.11 (GPIO20/U0RXD)
- net TX: now also R3.2; no longer U2.12 (GPIO21/U0TXD)
- net TXEN: now also R4.1; no longer U2.15 (GPIO3/ADC1_CH3)
- new net: R3.1, U2.12 (GPIO21/U0TXD)
- new net: R4.2, U2.15 (GPIO3/ADC1_CH3)
- new net: R2.1, U2.11 (GPIO20/U0RXD)
Changed lines of the file:
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@@
+    (stroke (width 0) (type default))
+  )
+  (wire (pts (xy 127 68.58) (xy 134.62 68.58))
     (stroke (width 0) (type default))
   )
@@
     (effects (font (size 1.27 1.27)) (justify right bottom))
   )
-  (label "TX" (at 189.23 63.5 0) (fields_autoplaced)
+  (label "TX" (at 196.85 63.5 0) (fields_autoplaced)
     (effects (font (size 1.27 1.27)) (justify left bottom))
   )
@@
     (effects (font (size 1.27 1.27)) (justify right bottom))
   )
-  (label "TXEN" (at 134.62 68.58 180) (fields_autoplaced)
-    (effects (font (size 1.27 1.27)) (justify right bottom))
-  )
-  (label "RX" (at 189.23 60.96 0) (fields_autoplaced)
+  (label "TXEN" (at 119.38 68.58 180) (fields_autoplaced)
+    (effects (font (size 1.27 1.27)) (justify right bottom))
+  )
+  (label "RX" (at 196.85 60.96 0) (fields_autoplaced)
     (effects (font (size 1.27 1.27)) (justify left bottom))
   )
@@
     (effects (font (size 1.27 1.27)) (justify left bottom))
   )
+  (symbol (lib_id "power:+5V") (at 104.14 120.65 0) (unit 1)
+    (in_bom yes) (on_board yes) (dnp no) (fields_autoplaced)
+    (property "Reference" "#PWR0102" (at 104.14 124.46 0)
+      (effects (font (size 1.27 1.27)) hide)
+    )
+    (property "Value" "+5V" (at 104.14 117.1671 0)
+      (effects (font (size 1.27 1.27)))
+    )
+    (property "Footprint" "" (at 104.14 120.65 0)
+      (effects (font (size 1.27 1.27)) hide)
+    )
+    (property "Datasheet" "" (at 104.14 120.65 0)
+      (effects (font (size 1.27 1.27)) hide)
+    )
+    (pin "1")
+    (instances
+      (project "vertical"
+        (path "/32f9e9f8-9d15-4d51-acc1-705de5fd2b71"
+          (reference "#PWR0102") (unit 1) (value "+5V") (footprint "")
+        )
+      )
+    )
+  )
   (symbol (lib_id "Device:C") (at 81.28 87.63 0) (unit 1)
     (in_bom yes) (on_board yes) (dnp no) (fields_autoplaced)
@@
     )
   )
+  (symbol (lib_id "Device:R") (at 193.04 63.5 90) (unit 1)
+    (in_bom yes) (on_board yes) (dnp no)
+    (property "Reference" "R3" (at 193.04 66.04 90)
+      (effects (font (size 1.27 1.27)))
+    )
+    (property "Value" "270R" (at 198.12 66.04 90)
+      (effects (font (size 1.27 1.27)))
+    )
+    (property "Footprint" "Resistor_SMD:R_0805_2012Metric_Pad1.20x1.40mm_HandSolder" (at 193.04 65.278 90)
+      (effects (font (size 1.27 1.27)) hide)
+    )
+    (property "Datasheet" "~" (at 193.04 63.5 0)
+      (effects (font (size 1.27 1.27)) hide)
+    )
+    (pin "1")
+    (pin "2")
+    (instances
+      (project "vertical"
+        (path "/32f9e9f8-9d15-4d51-acc1-705de5fd2b71"
+          (reference "R3") (unit 1) (value "270R") (footprint "Resistor_SMD:R_0805_2012Metric_Pad1.20x1.40mm_HandSolder")
+        )
+      )
+    )
+  )
   (symbol (lib_id "power:+3V3") (at 134.62 55.88 90) (unit 1)
     (in_bom yes) (on_board yes) (dnp no) (fields_autoplaced)
@@
       (effects (font (size 1.27 1.27)))
     )
-    (property "Footprint" "Connector_PinHeader_2.54mm:PinHeader_1x02_P2.54mm_Vertical" (at 233.68 111.76 0)
+    (property "Footprint" "LED_SMD:LED_2010_5025Metric" (at 233.68 111.76 0)
       (effects (font (size 1.27 1.27)) hide)
     )
@@
       (project "vertical"
         (path "/32f9e9f8-9d15-4d51-acc1-705de5fd2b71"
-          (reference "D1") (unit 1) (value "LED") (footprint "Connector_PinHeader_2.54mm:PinHeader_1x02_P2.54mm_Vertical")
-        )
-      )
-    )
-  )
-  (symbol (lib_id "power:+3V3") (at 104.14 120.65 0) (unit 1)
-    (in_bom yes) (on_board yes) (dnp no)
-    (property "Reference" "#PWR0101" (at 104.14 124.46 0)
-      (effects (font (size 1.27 1.27)) hide)
-    )
-    (property "Value" "+3V3" (at 104.14 117.1671 0)
-      (effects (font (size 1.27 1.27)))
-    )
-    (property "Footprint" "" (at 104.14 120.65 0)
-      (effects (font (size 1.27 1.27)) hide)
-    )
-    (property "Datasheet" "" (at 104.14 120.65 0)
-      (effects (font (size 1.27 1.27)) hide)
-    )
-    (pin "1")
-    (instances
-      (project "vertical"
-        (path "/32f9e9f8-9d15-4d51-acc1-705de5fd2b71"
-          (reference "#PWR0101") (unit 1) (value "+3V3") (footprint "")
+          (reference "D1") (unit 1) (value "LED") (footprint "LED_SMD:LED_2010_5025Metric")
         )
       )
@@
         (path "/32f9e9f8-9d15-4d51-acc1-705de5fd2b71"
           (reference "J2") (unit 1) (value "PROG") (footprint "Connector_PinHeader_2.54mm:PinHeader_1x03_P2.54mm_Vertical")
+        )
+      )
+    )
+  )
+  (symbol (lib_id "Device:R") (at 123.19 68.58 90) (unit 1)
+    (in_bom yes) (on_board yes) (dnp no)
+    (property "Reference" "R4" (at 123.19 66.04 90)
+      (effects (font (size 1.27 1.27)))
+    )
+    (property "Value" "270R" (at 128.27 66.04 90)
+      (effects (font (size 1.27 1.27)))
+    )
+    (property "Footprint" "Resistor_SMD:R_0805_2012Metric_Pad1.20x1.40mm_HandSolder" (at 123.19 70.358 90)
+      (effects (font (size 1.27 1.27)) hide)
+    )
+    (property "Datasheet" "~" (at 123.19 68.58 0)
+      (effects (font (size 1.27 1.27)) hide)
+    )
+    (pin "1")
+    (pin "2")
+    (instances
+      (project "vertical"
+        (path "/32f9e9f8-9d15-4d51-acc1-705de5fd2b71"
+          (reference "R4") (unit 1) (value "270R") (footprint "Resistor_SMD:R_0805_2012Metric_Pad1.20x1.40mm_HandSolder")
         )
       )
@@
     )
   )
+  (symbol (lib_id "Device:R") (at 193.04 60.96 90) (unit 1)
+    (in_bom yes) (on_board yes) (dnp no)
+    (property "Reference" "R2" (at 193.04 58.42 90)
+      (effects (font (size 1.27 1.27)))
+    )
+    (property "Value" "270R" (at 198.12 58.42 90)
+      (effects (font (size 1.27 1.27)))
+    )
+    (property "Footprint" "Resistor_SMD:R_0805_2012Metric_Pad1.20x1.40mm_HandSolder" (at 193.04 62.738 90)
+      (effects (font (size 1.27 1.27)) hide)
+    )
+    (property "Datasheet" "~" (at 193.04 60.96 0)
+      (effects (font (size 1.27 1.27)) hide)
+    )
+    (pin "1")
+    (pin "2")
+    (instances
+      (project "vertical"
+        (path "/32f9e9f8-9d15-4d51-acc1-705de5fd2b71"
+          (reference "R2") (unit 1) (value "270R") (footprint "Resistor_SMD:R_0805_2012Metric_Pad1.20x1.40mm_HandSolder")
+        )
+      )
+    )
+  )
   (symbol (lib_id "Connector:Conn_01x04_Male") (at 189.23 128.27 180) (unit 1)
     (in_bom yes) (on_board yes) (dnp no) (fields_autoplaced)
@@
       (effects (font (size 1.27 1.27)) (justify right))
     )
-    (property "Footprint" "Connector_PinHeader_2.54mm:PinHeader_1x04_P2.54mm_Vertical" (at 189.23 128.27 0)
+    (property "Footprint" "Connector_PinHeader_2.54mm:PinHeader_1x04_P2.54mm_Horizontal" (at 189.23 128.27 0)
       (effects (font (size 1.27 1.27)) hide)
     )
@@
       (project "vertical"
         (path "/32f9e9f8-9d15-4d51-acc1-705de5fd2b71"
-          (reference "J1") (unit 1) (value "internal") (footprint "Connector_PinHeader_2.54mm:PinHeader_1x04_P2.54mm_Vertical")
+          (reference "J1") (unit 1) (value "internal") (footprint "Connector_PinHeader_2.54mm:PinHeader_1x04_P2.54mm_Horizontal")
         )
       )
@@
   (symbol (lib_id "power:+5V") (at 49.53 82.55 90) (unit 1)
     (in_bom yes) (on_board yes) (dnp no) (fields_autoplaced)
-    (property "Reference" "#PWR0102" (at 53.34 82.55 0)
+    (property "Reference" "#PWR0101" (at 53.34 82.55 0)
       (effects (font (size 1.27 1.27)) hide)
     )
@@
       (project "vertical"
         (path "/32f9e9f8-9d15-4d51-acc1-705de5fd2b71"
-          (reference "#PWR0102") (unit 1) (value "+5V") (footprint "")
-        )
-      )
+          (reference "#PWR0101") (unit 1) (value "+5V") (footprint "")
+        )
+      )
