File: vertical/vertical.kicad_sch (KiCad schematic)
At the start: 14 parts, among them J1 internal, J2 PROG, U1 LM1117-3.3, U2 ESP32-C3-WROOM-02, U5 MAX485E

Commit message: WIP
Connections:
- net +5V: now also J1.1 (Pin_1); no longer J1.4 (Pin_4)
- net GND: now also J1.4 (Pin_4); no longer J1.1 (Pin_1)
- net RS485_A: now also J1.3 (Pin_3); no longer J1.2 (Pin_2)
- net RS485_B: now also J1.2 (Pin_2); no longer J1.3 (Pin_3)
Other:
- moved on the sheet: J1
Changed lines of the file:
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@@
-(kicad_sch (version 20221004) (generator eeschema)
+(kicad_sch (version 20221206) (generator eeschema)
   (paper "A4")
   (junction (at 81.28 82.55) (diameter 0) (color 0 0 0 0)
@@
       (project "vertical"
         (path "/32f9e9f8-9d15-4d51-acc1-705de5fd2b71"
-          (reference "#PWR0102") (unit 1) (value "+5V") (footprint "")
+          (reference "#PWR0102") (unit 1)
         )
       )
@@
       (project "vertical"
         (path "/32f9e9f8-9d15-4d51-acc1-705de5fd2b71"
-          (reference "C2") (unit 1) (value "47u") (footprint "Capacitor_SMD:C_0805_2012Metric_Pad1.18x1.45mm_HandSolder")
+          (reference "C2") (unit 1)
         )
       )
@@
       (project "vertical"
         (path "/32f9e9f8-9d15-4d51-acc1-705de5fd2b71"
-          (reference "C1") (unit 1) (value "10u") (footprint "Capacitor_SMD:C_0805_2012Metric_Pad1.18x1.45mm_HandSolder")
+          (reference "C1") (unit 1)
         )
       )
@@
       (project "vertical"
         (path "/32f9e9f8-9d15-4d51-acc1-705de5fd2b71"
-          (reference "C3") (unit 1) (value "47u") (footprint "Capacitor_SMD:C_0805_2012Metric_Pad1.18x1.45mm_HandSolder")
+          (reference "C3") (unit 1)
         )
       )
@@
       (project "vertical"
         (path "/32f9e9f8-9d15-4d51-acc1-705de5fd2b71"
-          (reference "R3") (unit 1) (value "270R") (footprint "Resistor_SMD:R_0805_2012Metric_Pad1.20x1.40mm_HandSolder")
+          (reference "R3") (unit 1)
         )
       )
@@
       (project "vertical"
         (path "/32f9e9f8-9d15-4d51-acc1-705de5fd2b71"
-          (reference "#PWR01") (unit 1) (value "+3V3") (footprint "")
+          (reference "#PWR01") (unit 1)
         )
       )
@@
       (project "vertical"
         (path "/32f9e9f8-9d15-4d51-acc1-705de5fd2b71"
-          (reference "D1") (unit 1) (value "LED") (footprint "LED_SMD:LED_2010_5025Metric")
+          (reference "D1") (unit 1)
         )
       )
@@
       (project "vertical"
         (path "/32f9e9f8-9d15-4d51-acc1-705de5fd2b71"
-          (reference "U5") (unit 1) (value "MAX485E") (footprint "Package_SO:SO-8_3.9x4.9mm_P1.27mm")
+          (reference "U5") (unit 1)
         )
       )
@@
       (project "vertical"
         (path "/32f9e9f8-9d15-4d51-acc1-705de5fd2b71"
-          (reference "#PWR05") (unit 1) (value "GND") (footprint "")
+          (reference "#PWR05") (unit 1)
         )
       )
@@
       (project "vertical"
         (path "/32f9e9f8-9d15-4d51-acc1-705de5fd2b71"
-          (reference "U1") (unit 1) (value "LM1117-3.3") (footprint "Package_TO_SOT_SMD:SOT-223-3_TabPin2")
+          (reference "U1") (unit 1)
         )
       )
@@
       (project "vertical"
         (path "/32f9e9f8-9d15-4d51-acc1-705de5fd2b71"
-          (reference "R1") (unit 1) (value "270R") (footprint "Resistor_SMD:R_0805_2012Metric_Pad1.20x1.40mm_HandSolder")
+          (reference "R1") (unit 1)
         )
       )
@@
       (project "vertical"
         (path "/32f9e9f8-9d15-4d51-acc1-705de5fd2b71"
-          (reference "J2") (unit 1) (value "PROG") (footprint "Connector_PinHeader_2.54mm:PinHeader_1x03_P2.54mm_Vertical")
+          (reference "J2") (unit 1)
         )
       )
@@
       (project "vertical"
         (path "/32f9e9f8-9d15-4d51-acc1-705de5fd2b71"
-          (reference "R4") (unit 1) (value "270R") (footprint "Resistor_SMD:R_0805_2012Metric_Pad1.20x1.40mm_HandSolder")
+          (reference "R4") (unit 1)
         )
       )
@@
       (project "vertical"
         (path "/32f9e9f8-9d15-4d51-acc1-705de5fd2b71"
-          (reference "U2") (unit 1) (value "ESP32-C3-WROOM-02") (footprint "Espressif:ESP32-C3-WROOM-02")
+          (reference "U2") (unit 1)
         )
       )
@@
       (project "vertical"
         (path "/32f9e9f8-9d15-4d51-acc1-705de5fd2b71"
-          (reference "#PWR04") (unit 1) (value "+3V3") (footprint "")
+          (reference "#PWR04") (unit 1)
         )
       )
@@
       (project "vertical"
         (path "/32f9e9f8-9d15-4d51-acc1-705de5fd2b71"
-          (reference "#PWR0107") (unit 1) (value "GND") (footprint "")
+          (reference "#PWR0107") (unit 1)
         )
       )
@@
       (project "vertical"
         (path "/32f9e9f8-9d15-4d51-acc1-705de5fd2b71"
-          (reference "R2") (unit 1) (value "270R") (footprint "Resistor_SMD:R_0805_2012Metric_Pad1.20x1.40mm_HandSolder")
-        )
-      )
-    )
-  )
-  (symbol (lib_id "Connector:Conn_01x04_Male") (at 189.23 128.27 180) (unit 1)
-    (in_bom yes) (on_board yes) (dnp no) (fields_autoplaced)
-    (property "Reference" "J1" (at 189.9412 126.4055 0)
+          (reference "R2") (unit 1)
+        )
+      )
+    )
+  )
+  (symbol (lib_id "Connector:Conn_01x04_Male") (at 189.23 125.73 0) (mirror y) (unit 1)
+    (in_bom yes) (on_board yes) (dnp no)
+    (property "Reference" "J1" (at 189.9412 127.5945 0)
       (effects (font (size 1.27 1.27)) (justify right))
     )
-    (property "Value" "internal" (at 189.9412 128.1677 0)
+    (property "Value" "internal" (at 189.9412 125.8323 0)
       (effects (font (size 1.27 1.27)) (justify right))
     )
-    (property "Footprint" "Connector_PinHeader_2.54mm:PinHeader_1x04_P2.54mm_Horizontal" (at 189.23 128.27 0)
-      (effects (font (size 1.27 1.27)) hide)
-    )
-    (property "Datasheet" "~" (at 189.23 128.27 0)
+    (property "Footprint" "Connector_PinHeader_2.54mm:PinHeader_1x04_P2.54mm_Horizontal" (at 189.23 125.73 0)
+      (effects (font (size 1.27 1.27)) hide)
+    )
+    (property "Datasheet" "~" (at 189.23 125.73 0)
       (effects (font (size 1.27 1.27)) hide)
     )
@@
       (project "vertical"
         (path "/32f9e9f8-9d15-4d51-acc1-705de5fd2b71"
-          (reference "J1") (unit 1) (value "internal") (footprint "Connector_PinHeader_2.54mm:PinHeader_1x04_P2.54mm_Horizontal")
+          (reference "J1") (unit 1)
         )
       )
@@
       (project "vertical"
         (path "/32f9e9f8-9d15-4d51-acc1-705de5fd2b71"
-          (reference "#PWR0105") (unit 1) (value "GND") (footprint "")
+          (reference "#PWR0105") (unit 1)
         )
       )
@@
       (project "vertical"
         (path "/32f9e9f8-9d15-4d51-acc1-705de5fd2b71"
-          (reference "C8") (unit 1) (value "100n") (footprint "Capacitor_SMD:C_0805_2012Metric_Pad1.18x1.45mm_HandSolder")
+          (reference "C8") (unit 1)
         )
       )
@@
       (project "vertical"
         (path "/32f9e9f8-9d15-4d51-acc1-705de5fd2b71"
-          (reference "#PWR0104") (unit 1) (value "GND") (footprint "")
+          (reference "#PWR0104") (unit 1)
         )
       )
@@
       (project "vertical"
         (path "/32f9e9f8-9d15-4d51-acc1-705de5fd2b71"
-          (reference "#PWR02") (unit 1) (value "+3V3") (footprint "")
+          (reference "#PWR02") (unit 1)
         )
       )
@@
       (project "vertical"
         (path "/32f9e9f8-9d15-4d51-acc1-705de5fd2b71"
-          (reference "#PWR0101") (unit 1) (value "+5V") (footprint "")
+          (reference "#PWR0101") (unit 1)
         )
       )
@@
       (project "vertical"
         (path "/32f9e9f8-9d15-4d51-acc1-705de5fd2b71"
-          (reference "#PWR0103") (unit 1) (value "GND") (footprint "")
+          (reference "#PWR0103") (unit 1)
         )
       )
@@
   )
   (sheet_instances
-    (path "/32f9e9f8-9d15-4d51-acc1-705de5fd2b71" (page "1"))
+    (path "/" (page "1"))
   )
 )

Commit message: board update
Parts:
- removed R2, R4: 270R, Resistor_SMD:R_0805_2012Metric_Pad1.20x1.40mm_HandSolder, symbol Device:R
- added C4: 1u, Capacitor_SMD:C_0805_2012Metric_Pad1.18x1.45mm_HandSolder, symbol Device:C
- added D2: BAT54S, Package_TO_SOT_SMD:SOT-23, symbol Diode:BAT54S
- added R5: 10k, Resistor_SMD:R_0805_2012Metric_Pad1.20x1.40mm_HandSolder, symbol Device:R
- D1: now not fitted
- J1: symbol Connector:Conn_01x04_Male -> Connector_Generic:Conn_01x04; now not fitted
- J2: symbol Connector:Conn_01x03_Female -> Connector_Generic:Conn_01x03
- R3: value 270R -> 1k5
- U1: symbol Regulator_Linear:LM1117-3.3 -> Regulator_Linear:LM1117MP-3.3
- U2: footprint Espressif:ESP32-C3-WROOM-02 -> Drake:ESP32-C3-WROOM-02-Handsolder
- U5: footprint Package_SO:SO-8_3.9x4.9mm_P1.27mm -> Package_SO:SOIC-8_3.9x4.9mm_P1.27mm
Connections:
- net +3V3: now also D2.2 (K), R5.1; no longer U2.2 (EN/CHIP_PU)
- net GND: now also C4.2, D2.1 (A)
- net RX: now also R3.2
- net TX: now also U2.12 (GPIO21/U0TXD); no longer R3.2
- net TXEN: now also U2.15 (GPIO3/ADC1_CH3)
- net USB_D+: now also J2.3 (Pin_3); no longer J2.1 (Pin_1)
- net USB_D-: now also J2.1 (Pin_1); no longer J2.3 (Pin_3)
- net at R3.1: now also U2.11 (GPIO20/U0RXD), D2.3 (COM); no longer U2.12 (GPIO21/U0TXD)
- new net: C4.1, R5.2, U2.2 (EN/CHIP_PU)
Other:
- moved on the sheet: R3

Commit message: Update KiCad design files
Parts:
- removed J2: PROG, Connector_PinHeader_2.54mm:PinHeader_1x03_P2.54mm_Vertical, symbol Connector_Generic:Conn_01x03
- removed R5: 10k, Resistor_SMD:R_0805_2012Metric_Pad1.20x1.40mm_HandSolder, symbol Device:R
- removed U2: ESP32-C3-WROOM-02, Drake:ESP32-C3-WROOM-02-Handsolder, symbol Espressif:ESP32-C3-WROOM-02
- added A1: 31mm, Drake:Wire antena 2.4GHz, symbol Device:Antenna
- added C5: 100n, Capacitor_SMD:C_0805_2012Metric, symbol Device:C
- added C6: 10u, Capacitor_SMD:C_0805_2012Metric, symbol Device:C
- added J1: DBG, Connector_PinHeader_2.54mm:PinHeader_1x01_P2.54mm_Vertical, symbol Connector_Generic:Conn_01x01
- added U2: PAN2110P0AA, Package_SO:SOIC-8_3.9x4.9mm_P1.27mm, symbol Drake:PAN2110P0AA
- added U3: PY32F003W1xSx, Package_SO:SOIC-16_3.9x9.9mm_P1.27mm, symbol MCU_Puya_PY32F:PY32F003W1xSx
- added X1: SWD, Drake:SWD, symbol Drake:SWD
- added Y1: 16MHz, Crystal:Crystal_SMD_3225-4Pin_3.2x2.5mm, symbol Device:Crystal_GND24_Small
- C1: value 10u -> 100n; footprint Capacitor_SMD:C_0805_2012Metric_Pad1.18x1.45mm_HandSolder -> Capacitor_SMD:C_0805_2012Metric
- C2: value 47u -> 100n; footprint Capacitor_SMD:C_0805_2012Metric_Pad1.18x1.45mm_HandSolder -> Capacitor_SMD:C_0805_2012Metric
- C3: value 47u -> 10u; footprint Capacitor_SMD:C_0805_2012Metric_Pad1.18x1.45mm_HandSolder -> Capacitor_SMD:C_0805_2012Metric
- C4: footprint Capacitor_SMD:C_0805_2012Metric_Pad1.18x1.45mm_HandSolder -> Capacitor_SMD:C_0805_2012Metric
- C7: renamed from C8; footprint Capacitor_SMD:C_0805_2012Metric_Pad1.18x1.45mm_HandSolder -> Capacitor_SMD:C_0805_2012Metric
- R1: renamed from R3; footprint Resistor_SMD:R_0805_2012Metric_Pad1.20x1.40mm_HandSolder -> Resistor_SMD:R_0805_2012Metric
- R2: renamed from R1; value 270R -> 330R; footprint Resistor_SMD:R_0805_2012Metric_Pad1.20x1.40mm_HandSolder -> Resistor_SMD:R_0805_2012Metric
- U1: value LM1117-3.3 -> LM1117MP-3.3
- renumbered D2 to D1, D1 to D2, J1 to J2, U5 to U4
Connections:
- net +3V3: now also C1.1, C4.1, C5.1, C6.1, U2.4 (VDD), U3.1 (VSS); no longer C2.1, C3.1
- net +5V: now also C3.1; no longer C1.1
- net GND: now also C5.2, C6.2, U2.7 (VSS), U3.16 (VCC), X1.2 (GND), Y1.2 (G), Y1.4 (G)
- net LED: now also U3.14 (PB0)
- net RS485_RX: now reaches D1.3 (COM), R1.1
- net RS485_RX: now also U3.9 (PA3)
- net RX: no longer names the net of R1.2, U4.1 (RO)
- net TX renamed RS485_TX
- net RS485_TX: now also U3.6 (PA0)
- net TXEN renamed RS485_TXEN
- net RS485_TXEN: now also U3.11 (PA5)
- new net: U2.5 (XC1), Y1.1
- new net: U2.6 (XC0), Y1.3
- new net: A1.1 (A), U2.8 (ANT)
- new net: C2.1, U3.5 (PF0/PF2-NRST)
- new net DEBUG: J1.1 (Pin_1), U3.13 (PA7)
- new net RF_DATA: U2.3 (SDA/DATA), U3.7 (PA1)
- new net RF_SCK: U2.2 (SCL/SCK), U3.8 (PA2)
- new net SWCLK: U3.4 (PF1/PA14-SWC), X1.3 (SWCLK)
- new net SWDIO: U3.3 (PA13-SWD), X1.1 (SWDIO)
- new net ~{RF_CS}: U2.1 (CSN), U3.10 (PA4)
- no-connect marks 9 -> 3
Other:
- moved on the sheet: C7, D1, D2, J2, R1, R2, U4
