File: board/bleriot-rs485.kicad_pcb (KiCad board)
At the start: 2 copper layers, 26 x 27 mm, 20 parts, among them J1 DBG, J2 internal, U1 LM1117MP-3.3, U2 PAN2110P0AA, U3 PY32F003W1xSx, U4 MAX485E, X1 SWD, Y1 16MHz

Commit message: dir layout
Connections:
- U3 pad 1: +3V3 -> GND
- U3 pad 16: GND -> +3V3
Routing:
- net +3V3: track 48.9 -> 52.9 mm, vias 1 -> 3
- net GND: vias 16 -> 22
Changed lines of the file:
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@@
 		(property ki_fp_filters "Crystal*")
 		(sheetname "/")
-		(sheetfile "vertical.kicad_sch")
+		(sheetfile "bleriot-rs485.kicad_sch")
 		(attr smd)
 		(fp_line
@@
 		(property ki_fp_filters "C_*")
 		(sheetname "/")
-		(sheetfile "vertical.kicad_sch")
+		(sheetfile "bleriot-rs485.kicad_sch")
 		(attr smd)
 		(fp_line
@@
 		)
 		(sheetname "/")
-		(sheetfile "vertical.kicad_sch")
+		(sheetfile "bleriot-rs485.kicad_sch")
 		(attr through_hole)
 		(fp_line
@@
 		(property ki_fp_filters "C_*")
 		(sheetname "/")
-		(sheetfile "vertical.kicad_sch")
+		(sheetfile "bleriot-rs485.kicad_sch")
 		(attr smd)
 		(fp_line
@@
 		(property ki_fp_filters "C_*")
 		(sheetname "/")
-		(sheetfile "vertical.kicad_sch")
+		(sheetfile "bleriot-rs485.kicad_sch")
 		(attr smd)
 		(fp_line
@@
 		)
 		(sheetname "/")
-		(sheetfile "vertical.kicad_sch")
+		(sheetfile "bleriot-rs485.kicad_sch")
 		(attr smd)
 		(fp_line
@@
 		(property ki_fp_filters "SOT?223*")
 		(sheetname "/")
-		(sheetfile "vertical.kicad_sch")
+		(sheetfile "bleriot-rs485.kicad_sch")
 		(attr smd)
 		(fp_line
@@
 		(property ki_fp_filters "C_*")
 		(sheetname "/")
-		(sheetfile "vertical.kicad_sch")
+		(sheetfile "bleriot-rs485.kicad_sch")
 		(attr smd)
 		(fp_line
@@
 		)
 		(sheetname "/")
-		(sheetfile "vertical.kicad_sch")
+		(sheetfile "bleriot-rs485.kicad_sch")
 		(attr smd)
 		(fp_line
@@
 			(layers "F.Cu" "F.Mask" "F.Paste")
 			(roundrect_rratio 0.25)
-			(net 3 "+3V3")
+			(net 2 "GND")
 			(pinfunction "VSS")
 			(pintype "power_in")
@@
 			(layers "F.Cu" "F.Mask" "F.Paste")
 			(roundrect_rratio 0.25)
-			(net 2 "GND")
+			(net 3 "+3V3")
 			(pinfunction "VCC")
 			(pintype "power_in")
@@
 		(property ki_fp_filters "Connector*:*_1x??_*")
 		(sheetname "/")
-		(sheetfile "vertical.kicad_sch")
+		(sheetfile "bleriot-rs485.kicad_sch")
 		(attr through_hole)
 		(fp_line
@@
 		)
 		(sheetname "/")
-		(sheetfile "vertical.kicad_sch")
+		(sheetfile "bleriot-rs485.kicad_sch")
 		(attr through_hole)
 		(fp_text user "${REFERENCE}"
@@
 		(property ki_fp_filters "C_*")
 		(sheetname "/")
-		(sheetfile "vertical.kicad_sch")
+		(sheetfile "bleriot-rs485.kicad_sch")
 		(attr smd)
 		(fp_line
@@
 		(property ki_fp_filters "C_*")
 		(sheetname "/")
-		(sheetfile "vertical.kicad_sch")
+		(sheetfile "bleriot-rs485.kicad_sch")
 		(attr smd)
 		(fp_line
@@
 		(property ki_fp_filters "R_*")
 		(sheetname "/")
-		(sheetfile "vertical.kicad_sch")
+		(sheetfile "bleriot-rs485.kicad_sch")
 		(attr smd)
 		(fp_line
@@
 		(property ki_fp_filters "Connector*:*_1x??_*")
 		(sheetname "/")
-		(sheetfile "vertical.kicad_sch")
+		(sheetfile "bleriot-rs485.kicad_sch")
 		(attr through_hole dnp)
 		(fp_line
@@
 		(property ki_fp_filters "C_*")
 		(sheetname "/")
-		(sheetfile "vertical.kicad_sch")
+		(sheetfile "bleriot-rs485.kicad_sch")
 		(attr smd)
 		(fp_line
@@
 		(property ki_fp_filters "LED* LED_SMD:* LED_THT:*")
 		(sheetname "/")
-		(sheetfile "vertical.kicad_sch")
+		(sheetfile "bleriot-rs485.kicad_sch")
 		(attr smd dnp)
 		(fp_line
@@
 		(property ki_fp_filters "SOT?23*")
 		(sheetname "/")
-		(sheetfile "vertical.kicad_sch")
+		(sheetfile "bleriot-rs485.kicad_sch")
 		(attr smd)
 		(fp_line
@@
 		(property ki_fp_filters "R_*")
 		(sheetname "/")
-		(sheetfile "vertical.kicad_sch")
+		(sheetfile "bleriot-rs485.kicad_sch")
 		(attr smd)
 		(fp_line
@@
 		(property ki_fp_filters "DIP*W7.62mm* SOIC*3.9x4.9mm*P1.27mm*")
 		(sheetname "/")
-		(sheetfile "vertical.kicad_sch")
+		(sheetfile "bleriot-rs485.kicad_sch")
 		(attr smd)
 		(fp_line
@@
 	)
 	(via
+		(at 140 79)
+		(size 0.8)
+		(drill 0.4)
+		(layers "F.Cu" "B.Cu")
+		(free yes)
+		(net 2)
+	)
+	(via
 		(at 128 89)
 		(size 0.8)
@@
 	)
 	(via
+		(at 140 80)
+		(size 0.8)
+		(drill 0.4)
+		(layers "F.Cu" "B.Cu")
+		(free yes)
+		(net 2)
+	)
+	(via
 		(at 148.5 83)
 		(size 0.8)
@@
 	)
 	(via
+		(at 140 75)
+		(size 0.8)
+		(drill 0.4)
+		(layers "F.Cu" "B.Cu")
+		(free yes)
+		(net 2)
+	)
+	(via
 		(at 137 67)
 		(size 0.8)
@@
 	)
 	(via
+		(at 140 76)
+		(size 0.8)
+		(drill 0.4)
+		(layers "F.Cu" "B.Cu")
+		(free yes)
+		(net 2)
+	)
+	(via
 		(at 128.5 68)
 		(size 0.8)
@@
 	)
 	(via
+		(at 140 77)
+		(size 0.8)
+		(drill 0.4)
+		(layers "F.Cu" "B.Cu")
+		(free yes)
+		(net 2)
+	)
+	(via
 		(at 133 68)
 		(size 0.8)
@@
 	)
 	(via
+		(at 140 81)
+		(size 0.8)
+		(drill 0.4)
+		(layers "F.Cu" "B.Cu")
+		(free yes)
+		(net 2)
+	)
+	(via
 		(at 128.5 67)
 		(size 0.8)
@@
 	)
 	(segment
+		(start 133.495555 81.045555)
+		(end 134.45 82)
+		(width 0.4)
+		(layer "F.Cu")
+		(net 3)
+	)
+	(segment
 		(start 142.05 82.9)
 		(end 142.05 79)
@@
 	)
 	(segment
+		(start 129.525 79.445)
+		(end 129.525 80.525)
+		(width 0.4)
+		(layer "F.Cu")
+		(net 3)
+	)
+	(segment
 		(start 134.45 84.5)
 		(end 134.45 82)
@@
 	)
 	(segment
-		(start 134.45 82)
-		(end 134.45 79.47)
-		(width 1)
+		(start 134.45 84.5)
+		(end 133.45 85.5)
+		(width 0.4)
 		(layer "F.Cu")
 		(net 3)
 	)
 	(segment
-		(start 134.45 84.5)
-		(end 133.45 85.5)
+		(start 133.45 85.5)
+		(end 133.45 88.05)
 		(width 0.4)
 		(layer "F.Cu")
@@
 	)
 	(segment
-		(start 134.45 79.47)
-		(end 134.475 79.445)
+		(start 142.05 74.38)
+		(end 142.525 73.905)
 		(width 1)
 		(layer "F.Cu")
@@
 	)
 	(segment
-		(start 133.45 85.5)
-		(end 133.45 88.05)
+		(start 129.525 80.525)
+		(end 129.75 80.75)
 		(width 0.4)
 		(layer "F.Cu")
@@
 	)
 	(segment
-		(start 142.05 74.38)
-		(end 142.525 73.905)
-		(width 1)
+		(start 133.495555 81.036011)
+		(end 133.495555 81.045555)
+		(width 0.4)
 		(layer "F.Cu")
 		(net 3)
@@
 	)
 	(via
+		(at 129.75 80.75)
+		(size 0.8)
+		(drill 0.4)
+		(layers "F.Cu" "B.Cu")
+		(net 3)
+	)
+	(via
+		(at 133.495555 81.036011)
+		(size 0.8)
+		(drill 0.4)
+		(layers "F.Cu" "B.Cu")
+		(net 3)
+	)
+	(via
 		(at 126 82)
 		(size 0.8)
@@
 		(width 0.4)
 		(layer "B.Cu")
+		(net 3)
+	)
+	(segment
+		(start 129.75 80.75)
+		(end 130.036011 81.036011)
+		(width 0.4)
+		(layer "B.Cu")
+		(net 3)
+	)
+	(segment
+		(start 130.036011 81.036011)
+		(end 133.495555 81.036011)
+		(width 0.4)
+		(layer "B.Cu")

Commit message: WIP
Parts:
- removed A1: 31mm, Drake:Wire antena 2.4GHz
- removed C1, C2, C5: 100n, Capacitor_SMD:C_0805_2012Metric
- removed C4: 1u, Capacitor_SMD:C_0805_2012Metric
- removed D2: LED, LED_SMD:LED_2010_5025Metric
- removed J1: DBG, Connector_PinHeader_2.54mm:PinHeader_1x01_P2.54mm_Vertical
- removed J2: internal, Connector_PinHeader_2.54mm:PinHeader_1x04_P2.54mm_Horizontal
- removed R2: 330R, Resistor_SMD:R_0805_2012Metric
- removed U2: PAN2110P0AA, Package_SO:SOIC-8_3.9x4.9mm_P1.27mm
- removed U3: PY32F003W1xSx, Package_SO:SOIC-16_3.9x9.9mm_P1.27mm
- removed X1: SWD, Drake:SWD
- removed Y1: 16MHz, Crystal:Crystal_SMD_3225-4Pin_3.2x2.5mm
- added A2: Antenna_Shield, RF_Antenna:Texas_SWRA117D_2.4GHz_Right, F.Cu at (153.1, 36.6)
- added C10: 1u, Capacitor_SMD:C_0805_2012Metric, F.Cu at (144.9, 54.0)
- added C11: 100n, Capacitor_SMD:C_0805_2012Metric, F.Cu at (144.9, 50.0)
- added C12: 100n, Capacitor_SMD:C_0805_2012Metric, F.Cu at (147.9, 54.0)
- added C8: 1u, Capacitor_SMD:C_0805_2012Metric, F.Cu at (161.0, 45.0)
- added C9: 100n, Capacitor_SMD:C_0805_2012Metric, F.Cu at (159.0, 45.0)
- added D3: WS2812B, LED_SMD:LED_WS2812B_PLCC4_5.0x5.0mm_P3.2mm, F.Cu at (146.0, 43.0)
- added D4: LED, LED_SMD:LED_0805_2012Metric_Pad1.15x1.40mm_HandSolder, F.Cu at (146.0, 43.0)
- added H1: MountingHole, MountingHole:MountingHole_3.7mm_Pad_Via, F.Cu at (62.3, 38.3)
- added J3: POWER, Connector_Phoenix_MSTB:PhoenixContact_MSTBA_2,5_2-G_1x02_P5.00mm_Horizontal, F.Cu at (172.0, 60.2)
- added J4: RS485, Connector_Phoenix_MSTB:PhoenixContact_MSTBA_2,5_3-G_1x03_P5.00mm_Horizontal, F.Cu at (146.0, 60.2)
- added R3: 10k, Resistor_SMD:R_0805_2012Metric, F.Cu at (151.0, 45.0)
- added R4: 330R, Resistor_SMD:R_0805_2012Metric, F.Cu at (151.0, 41.0)
- added U5: PAN2110P0AA, Package_SO:SOIC-8_3.9x4.9mm_P1.27mm, F.Cu at (155.0, 42.0)
- added U6: PY32F030F1xPx, Package_SO:TSSOP-20_4.4x6.5mm_P0.65mm, F.Cu at (153.9, 51.0)
- added X2: SWD, Drake:SWD, F.Cu at (164.0, 63.0)
- added Y2: 16MHz, Crystal:Crystal_SMD_3225-4Pin_3.2x2.5mm, F.Cu at (160.0, 41.0)
- C7, D1, R1, U4: moved to F.Cu
- moved C3 56.3 mm to (177.0, 51.0), turned to -90 degrees
- moved C6 56.1 mm to (169.0, 41.0)
- moved C7 55.3 mm to (174.0, 51.0), turned to -90 degrees
- moved U1 53.2 mm to (175.0, 44.0), turned to 90 degrees
- moved D1 53.0 mm to (167.0, 46.0), turned to 180 degrees
- moved U4 44.9 mm to (168.0, 52.0), turned to 0 degrees
- moved R1 43.6 mm to (161.0, 50.0), turned to 0 degrees
Routing:
- net +3V3: track 52.9 -> 139.0 mm, vias 3 -> 0
- net /RS485_B: track 3.59 -> 25.5 mm
- net Net-(U6-PA11): track 0.00 -> 17.3 mm, vias 0 -> 1
- net /RS485_A: track 3.99 -> 21.0 mm
- net Net-(U6-PA13): track 0.00 -> 13.2 mm, vias 0 -> 1
- net Net-(U3-PF0/PF2-NRST): track 12.9 -> 0.00 mm, vias 2 -> 0
- net /LED: track 19.1 -> 6.69 mm, vias 1 -> 0
- net /~{RF_CS}: track 18.1 -> 9.04 mm
- net Net-(D4-K): track 0.00 -> 9.00 mm, vias 0 -> 2
- net +5V: track 14.0 -> 22.3 mm
- net Net-(U5-XC0): track 0.00 -> 7.26 mm
- net /RS485_RX: track 23.4 -> 17.0 mm, vias 1 -> 0
- net Net-(U6-PF2-NRST): track 0.00 -> 6.27 mm
- net Net-(U2-XC1): track 5.68 -> 0.00 mm
- net Net-(U2-XC0): track 5.22 -> 0.00 mm
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Other:
- board size 26 x 27 mm -> 40 x 42 mm
- board text added: "+5V"
- board text added: "A"
- board text added: "B"
- board text added: "GND"
- board text added: "bleriot-rs485 v1.0 drake.cz"
- board text removed: "RS485 WiFi v2.2 drake.cz"

Commit message: WIP
Parts:
- removed H1: MountingHole, MountingHole:MountingHole_3.7mm_Pad_Via

Commit message: WIP
Parts:
- J3: footprint Connector_Phoenix_MSTB:PhoenixContact_MSTBA_2,5_2-G_1x02_P5.00mm_Horizontal -> Connector_Phoenix_MC:PhoenixContact_MC_1,5_2-G-3.5_1x02_P3.50mm_Horizontal
- J4: footprint Connector_Phoenix_MSTB:PhoenixContact_MSTBA_2,5_3-G_1x03_P5.00mm_Horizontal -> Connector_Phoenix_MC:PhoenixContact_MC_1,5_3-G-3.5_1x03_P3.50mm_Horizontal
- moved J4 3.57 mm to (149.1, 62.1)
- moved J3 2.87 mm to (169.8, 62.1)
- moved X2 2.50 mm to (161.5, 63.0)
- moved D3 0.50 mm to (146.5, 43.0)
- moved D4 0.50 mm to (146.5, 43.0)
Routing:
- net +5V: track 22.3 -> 25.7 mm
- net /RS485_A: track 21.0 -> 22.9 mm
- net /RS485_B: track 25.5 -> 26.7 mm
- net Net-(U6-PA11): track 17.3 -> 16.3 mm
- net Net-(U6-PA13): track 13.2 -> 12.2 mm
- net Net-(D4-K): track 9.00 -> 9.50 mm
- net GND: vias 43 -> 41
Other:
- outline, holes or cut-outs redrawn

Commit message: board fixes
Parts:
- removed D1: BAT54S, Package_TO_SOT_SMD:SOT-23
- removed R1: 1k5, Resistor_SMD:R_0805_2012Metric
- U4: value MAX485E -> ST3485EBDR
Connections:
- C7 pad 1: +5V -> +3V3
- U4 pad 1: Net-(U4-RO) -> /RS485_RX
- U4 pad 8: +5V -> +3V3
- U6 pad 13: Net-(U6-PA11) -> unconnected-(U6-PA11-Pad13)
- U6 pad 15: unconnected-(U6-PA14-Pad15) -> Net-(U6-PA14)
- X2 pad 1: Net-(U6-PA11) -> Net-(U6-PA13)
- X2 pad 3: Net-(U6-PA13) -> Net-(U6-PA14)
Routing:
- net Net-(U6-PA11): track 16.3 -> 0.00 mm, vias 1 -> 0
- net Net-(U6-PA14): track 0.00 -> 12.4 mm, vias 0 -> 1
- net +5V: track 25.7 -> 19.2 mm
- net +3V3: track 139.3 -> 145.2 mm
- net Net-(U6-PA13): track 12.2 -> 16.6 mm
- net /RS485_RX: track 17.0 -> 13.2 mm
- net Net-(U4-RO): track 3.65 -> 0.00 mm
- net /RS485_TXEN: track 12.3 -> 11.4 mm
- net GND: vias 41 -> 51
Other:
- board text added: "bleriot-rs485 v1.1 drake.cz"
- board text removed: "bleriot-rs485 v1.0 drake.cz"
