File: board/bleriot-rs485.kicad_sch (KiCad schematic)
At the start: 20 parts, among them J1 DBG, J2 internal, U1 LM1117MP-3.3, U2 PAN2110P0AA, U3 PY32F003W1xSx, U4 MAX485E, X1 SWD, Y1 16MHz

Commit message: dir layout
Connections:
- net +3V3: now also U3.16 (VCC); no longer U3.1 (VSS)
- net GND: now also U3.1 (VSS); no longer U3.16 (VCC)
Other:
- moved on the sheet: C1
Changed lines of the file:
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@@
 	)
 	(junction
-		(at 55.88 54.61)
+		(at 116.84 54.61)
 		(diameter 0)
 		(color 0 0 0 0)
@@
 	(wire
 		(pts
-			(xy 55.88 54.61) (xy 66.04 54.61)
+			(xy 116.84 54.61) (xy 106.68 54.61)
 		)
 		(stroke
@@
 	(wire
 		(pts
-			(xy 55.88 48.26) (xy 55.88 54.61)
+			(xy 116.84 48.26) (xy 116.84 54.61)
 		)
 		(stroke
@@
 	(wire
 		(pts
-			(xy 54.61 54.61) (xy 55.88 54.61)
+			(xy 118.11 54.61) (xy 116.84 54.61)
 		)
 		(stroke
@@
 	(symbol
 		(lib_id "power:GND")
-		(at 46.99 54.61 270)
+		(at 125.73 54.61 90)
+		(mirror x)
 		(unit 1)
 		(exclude_from_sim no)
@@
 		(dnp no)
 		(property "Reference" "#PWR01"
-			(at 40.64 54.61 0)
+			(at 132.08 54.61 0)
 			(effects
 				(font
@@
 		)
 		(property "Value" "GND"
-			(at 42.164 54.61 90)
+			(at 130.556 54.61 90)
 			(effects
 				(font
@@
 		)
 		(property "Footprint" ""
-			(at 46.99 54.61 0)
+			(at 125.73 54.61 0)
 			(effects
 				(font
@@
 		)
 		(property "Datasheet" ""
-			(at 46.99 54.61 0)
+			(at 125.73 54.61 0)
 			(effects
 				(font
@@
 		)
 		(property "Description" "Power symbol creates a global label with name \"GND\" , ground"
-			(at 46.99 54.61 0)
+			(at 125.73 54.61 0)
 			(effects
 				(font
@@
 	(symbol
 		(lib_id "power:+3.3V")
-		(at 55.88 48.26 0)
+		(at 116.84 48.26 0)
+		(mirror y)
 		(unit 1)
 		(exclude_from_sim no)
@@
 		(dnp no)
 		(property "Reference" "#PWR03"
-			(at 55.88 52.07 0)
+			(at 116.84 52.07 0)
 			(effects
 				(font
@@
 		)
 		(property "Value" "+3V3"
-			(at 55.88 42.926 90)
+			(at 116.84 42.926 90)
 			(effects
 				(font
@@
 		)
 		(property "Footprint" ""
-			(at 55.88 48.26 0)
+			(at 116.84 48.26 0)
 			(effects
 				(font
@@
 		)
 		(property "Datasheet" ""
-			(at 55.88 48.26 0)
+			(at 116.84 48.26 0)
 			(effects
 				(font
@@
 		)
 		(property "Description" "Power symbol creates a global label with name \"+3.3V\""
-			(at 55.88 48.26 0)
+			(at 116.84 48.26 0)
 			(effects
 				(font
@@
 	(symbol
 		(lib_id "Device:C")
-		(at 50.8 54.61 270)
+		(at 121.92 54.61 90)
+		(mirror x)
 		(unit 1)
 		(exclude_from_sim no)
@@
 		(dnp no)
 		(property "Reference" "C1"
-			(at 50.8 51.308 90)
+			(at 121.92 51.308 90)
 			(effects
 				(font
@@
 		)
 		(property "Value" "100n"
-			(at 50.8 58.166 90)
+			(at 121.92 58.166 90)
 			(effects
 				(font
@@
 		)
 		(property "Footprint" "Capacitor_SMD:C_0805_2012Metric"
-			(at 46.99 55.5752 0)
+			(at 125.73 55.5752 0)
 			(effects
 				(font
@@
 		)
 		(property "Datasheet" "~"
-			(at 50.8 54.61 0)
+			(at 121.92 54.61 0)
 			(effects
 				(font
@@
 		)
 		(property "Description" "Unpolarized capacitor"
-			(at 50.8 54.61 0)
+			(at 121.92 54.61 0)
 			(effects
 				(font
@@
 	(symbol
 		(lib_id "power:GND")
-		(at 106.68 54.61 90)
+		(at 66.04 54.61 270)
 		(mirror x)
 		(unit 1)
@@
 		(dnp no)
 		(property "Reference" "#PWR014"
-			(at 113.03 54.61 0)
+			(at 59.69 54.61 0)
 			(effects
 				(font
@@
 		)
 		(property "Value" "GND"
-			(at 111.76 54.61 90)
+			(at 60.96 54.61 90)
 			(effects
 				(font
@@
 		)
 		(property "Footprint" ""
-			(at 106.68 54.61 0)
+			(at 66.04 54.61 0)
 			(effects
 				(font
@@
 		)
 		(property "Datasheet" ""
-			(at 106.68 54.61 0)
+			(at 66.04 54.61 0)
 			(effects
 				(font
@@
 		)
 		(property "Description" "Power symbol creates a global label with name \"GND\" , ground"
-			(at 106.68 54.61 0)
+			(at 66.04 54.61 0)
 			(effects
 				(font

Commit message: WIP
Parts:
- removed A1: 31mm, Drake:Wire antena 2.4GHz, symbol Device:Antenna
- removed C1, C2, C5: 100n, Capacitor_SMD:C_0805_2012Metric, symbol Device:C
- removed C4: 1u, Capacitor_SMD:C_0805_2012Metric, symbol Device:C
- removed D2: LED, LED_SMD:LED_2010_5025Metric, symbol Device:LED
- removed J1: DBG, Connector_PinHeader_2.54mm:PinHeader_1x01_P2.54mm_Vertical, symbol Connector_Generic:Conn_01x01
- removed J2: internal, Connector_PinHeader_2.54mm:PinHeader_1x04_P2.54mm_Horizontal, symbol Connector_Generic:Conn_01x04
- removed R2: 330R, Resistor_SMD:R_0805_2012Metric, symbol Device:R
- removed U2: PAN2110P0AA, Package_SO:SOIC-8_3.9x4.9mm_P1.27mm, symbol Drake:PAN2110P0AA
- removed U3: PY32F003W1xSx, Package_SO:SOIC-16_3.9x9.9mm_P1.27mm, symbol MCU_Puya_PY32F:PY32F003W1xSx
- removed X1: SWD, Drake:SWD, symbol Drake:SWD
- removed Y1: 16MHz, Crystal:Crystal_SMD_3225-4Pin_3.2x2.5mm, symbol Device:Crystal_GND24_Small
- added A2: Antenna_Shield, RF_Antenna:Texas_SWRA117D_2.4GHz_Right, symbol Device:Antenna_Shield
- added C10, C8: 1u, Capacitor_SMD:C_0805_2012Metric, symbol Device:C
- added C11, C12, C9: 100n, Capacitor_SMD:C_0805_2012Metric, symbol Device:C
- added D3: WS2812B, LED_SMD:LED_WS2812B_PLCC4_5.0x5.0mm_P3.2mm, symbol LED:WS2812B
- added D4: LED, LED_SMD:LED_0805_2012Metric_Pad1.15x1.40mm_HandSolder, symbol Device:LED
- added H1: MountingHole, MountingHole:MountingHole_3.7mm_Pad_Via, symbol Mechanical:MountingHole
- added J3: POWER, Connector_Phoenix_MSTB:PhoenixContact_MSTBA_2,5_2-G_1x02_P5.00mm_Horizontal, symbol Connector:Conn_01x02_Pin
- added J4: RS485, Connector_Phoenix_MSTB:PhoenixContact_MSTBA_2,5_3-G_1x03_P5.00mm_Horizontal, symbol Connector:Conn_01x03_Pin
- added R3: 10k, Resistor_SMD:R_0805_2012Metric, symbol Device:R
- added R4: 330R, Resistor_SMD:R_0805_2012Metric, symbol Device:R
- added U5: PAN2110P0AA, Package_SO:SOIC-8_3.9x4.9mm_P1.27mm, symbol Drake:PAN2110P0AA
- added U6: PY32F030F1xPx, Package_SO:TSSOP-20_4.4x6.5mm_P0.65mm, symbol MCU_Puya_PY32F:PY32F030F1xPx
- added X2: SWD, Drake:SWD, symbol Drake:SWD
- added Y2: 16MHz, Crystal:Crystal_SMD_3225-4Pin_3.2x2.5mm, symbol Device:Crystal_GND24_Small
Connections:
- net +3V3: now also C10.1, C12.1, C8.1, C9.1, D3.1 (VDD), R3.2, U5.4 (VDD), U6.9 (VCC)
- net +5V: now also J3.2 (Pin_2)
- net GND: now also A2.2 (Shield), C10.2, C11.2, C12.2, C8.2, C9.2, D3.3 (VSS), J3.1 (Pin_1), J4.1 (Pin_1), R4.1, U5.7 (VSS), U6.7 (VSS), X2.2 (GND), Y2.2 (G), Y2.4 (G)
- net LED: now also D3.4 (DIN), D4.2 (A), U6.1 (PF0-OSCIN)
- net RF_DATA: now also U5.3 (SDA/DATA), U6.6 (PA3)
- net RF_SCK: now also U5.2 (SCL/SCK), U6.5 (PA2)
- net RS485_A: now also J4.3 (Pin_3)
- net RS485_B: now also J4.2 (Pin_2)
- net RS485_RX: now also U6.19 (PB7)
- net RS485_TX: now also U6.18 (PB6)
- net RS485_TXEN: now also U6.20 (PF4-BOOT0)
- net ~{RF_CS}: now also R3.1, U5.1 (CSN), U6.4 (PF3)
- new net: D4.1 (K), R4.2
- new net: U6.13 (PA11), X2.1 (SWDIO)
- new net: U6.14 (PA13), X2.3 (SWCLK)
- new net: C11.1, U6.3 (PF2-NRST)
- new net: A2.1 (A), U5.8 (ANT)
- new net: U5.5 (XC1), Y2.1
- new net: U5.6 (XC0), Y2.3
- no-connect marks 3 -> 9
Other:
- moved on the sheet: C3, C6, C7, D1, R1, U1, U4

Commit message: WIP
Parts:
- removed H1: MountingHole, MountingHole:MountingHole_3.7mm_Pad_Via, symbol Mechanical:MountingHole
Changed lines of the file:
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@@
-	)
-	(symbol
-		(lib_id "Mechanical:MountingHole")
-		(at 214.63 139.7 0)
-		(unit 1)
-		(body_style 1)
-		(exclude_from_sim no)
-		(in_bom yes)
-		(on_board yes)
-		(in_pos_files yes)
-		(dnp no)
-		(fields_autoplaced yes)
-		(property "Reference" "H1"
-			(at 217.17 139.1055 0)
-			(show_name no)
-			(do_not_autoplace no)
-			(effects
-				(font
-					(size 1.27 1.27)
-				)
-				(justify left)
-			)
-		)
-		(property "Value" "MountingHole"
-			(at 217.17 140.8677 0)
-			(show_name no)
-			(do_not_autoplace no)
-			(effects
-				(font
-					(size 1.27 1.27)
-				)
-				(justify left)
-			)
-		)
-		(property "Footprint" "MountingHole:MountingHole_3.7mm_Pad_Via"
-			(at 214.63 139.7 0)
-			(hide yes)
-			(show_name no)
-			(do_not_autoplace no)
-			(effects
-				(font
-					(size 1.27 1.27)
-				)
-			)
-		)
-		(property "Datasheet" ""
-			(at 214.63 139.7 0)
-			(hide yes)
-			(show_name no)
-			(do_not_autoplace no)
-			(effects
-				(font
-					(size 1.27 1.27)
-				)
-			)
-		)
-		(property "Description" "Mounting Hole without connection"
-			(at 214.63 139.7 0)
-			(hide yes)
-			(show_name no)
-			(do_not_autoplace no)
-			(effects
-				(font
-					(size 1.27 1.27)
-				)
-			)
-		)
-		(instances
-			(project "bleriot-rs485"
-				(path "/32f9e9f8-9d15-4d51-acc1-705de5fd2b71"
-					(reference "H1")
-					(unit 1)
-				)
-			)
-		)
 	)
 	(symbol

Commit message: WIP
Parts:
- J3: footprint Connector_Phoenix_MSTB:PhoenixContact_MSTBA_2,5_2-G_1x02_P5.00mm_Horizontal -> Connector_Phoenix_MC:PhoenixContact_MC_1,5_2-G-3.5_1x02_P3.50mm_Horizontal
- J4: footprint Connector_Phoenix_MSTB:PhoenixContact_MSTBA_2,5_3-G_1x03_P5.00mm_Horizontal -> Connector_Phoenix_MC:PhoenixContact_MC_1,5_3-G-3.5_1x03_P3.50mm_Horizontal
Changed lines of the file:
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@@
 			)
 		)
-		(property "Footprint" "Connector_Phoenix_MSTB:PhoenixContact_MSTBA_2,5_3-G_1x03_P5.00mm_Horizontal"
+		(property "Footprint" "Connector_Phoenix_MC:PhoenixContact_MC_1,5_3-G-3.5_1x03_P3.50mm_Horizontal"
 			(at 35.56 114.3 0)
 			(hide yes)
@@
 			)
 		)
-		(property "Footprint" "Connector_Phoenix_MSTB:PhoenixContact_MSTBA_2,5_2-G_1x02_P5.00mm_Horizontal"
+		(property "Footprint" "Connector_Phoenix_MC:PhoenixContact_MC_1,5_2-G-3.5_1x02_P3.50mm_Horizontal"
 			(at 34.29 135.89 0)
 			(hide yes)

Commit message: board fixes
Parts:
- removed D1: BAT54S, Package_TO_SOT_SMD:SOT-23, symbol Diode:BAT54S
- removed R1: 1k5, Resistor_SMD:R_0805_2012Metric, symbol Device:R
- U4: value MAX485E -> ST3485EBDR
Connections:
- net +3V3: now also C7.1, U4.8 (VCC)
- net +5V: no longer C7.1, U4.8 (VCC)
- net RS485_RX: now also U4.1 (RO)
- net at U6.13 (PA11): no longer X2.1 (SWDIO)
- net at U6.14 (PA13): now also X2.1 (DIO); no longer X2.3 (SWCLK)
- net at U6.15 (PA14): now also X2.3 (CLK)
